File: AICE/iCE40.sch (KiCad schematic (older format))
At the start: 5 parts

Commit message: Add files via upload
Parts:
- removed U?: W25Q128JVS, Package_SO:SOIC-8_5.23x5.23mm_P1.27mm, symbol Memory_Flash:W25Q128JVS
- added R? (x3): R, symbol Device:R
- added U?: W25Q, symbol w25q:W25Q
Connections:
- net labels added: Om_SPI0, Om_SPI1, Om_SPI2, Om_SPI3, Om_SPI4, Om_SPI[4,0], iCE_MISO, iCE_MOSI, iCE_SCLK, iCE_SS
- net labels removed: Om_SPI[3,0], SPI0, SPI1, SPI2, SPI3
- wire segments 9 -> 25
Changed lines of the file:
@@
 Wire Wire Line
 	1300 7550 1800 7550
-Text HLabel 2100 6900 0    50   BiDi ~ 0
-Om_SPI[3,0]
+Text HLabel 2100 6800 0    50   BiDi ~ 0
+Om_SPI[4,0]
 Wire Bus Line
-	2100 6900 2250 6900
-Entry Wire Line
-	2250 7450 2350 7550
+	2100 6800 2250 6800
 Entry Wire Line
 	2250 7350 2350 7450
@@
 Entry Wire Line
 	2250 7150 2350 7250
-Wire Wire Line
-	2350 7250 2850 7250
-Wire Wire Line
-	2350 7350 2850 7350
-Wire Wire Line
-	2350 7450 2850 7450
-Wire Wire Line
-	2350 7550 2850 7550
-Wire Bus Line
-	2250 6900 2250 7450
-Wire Bus Line
-	1200 6900 1200 7450
+Entry Wire Line
+	2250 7050 2350 7150
+Text Label 2350 7150 0    50   ~ 0
+Om_SPI0
 Text Label 2350 7250 0    50   ~ 0
-SPI0
+Om_SPI1
 Text Label 2350 7350 0    50   ~ 0
-SPI1
+Om_SPI2
 Text Label 2350 7450 0    50   ~ 0
-SPI2
-Text Label 2350 7550 0    50   ~ 0
-SPI3
+Om_SPI3
 Text Label 1300 7150 0    50   ~ 0
 COMM0
@@
 COMM4
 $Comp
-L Memory_Flash:W25Q128JVS U?
-U 1 1 5E904339
-P 9450 5200
-F 0 "U?" H 9450 5781 50  0000 C CNN
-F 1 "W25Q128JVS" H 9450 5690 50  0000 C CNN
-F 2 "Package_SO:SOIC-8_5.23x5.23mm_P1.27mm" H 9450 5200 50  0001 C CNN
-F 3 "http://www.winbond.com/resource-files/w25q128jv_dtr%20revc%2003272018%20plus.pdf" H 9450 5200 50  0001 C CNN
-	1    9450 5200
+L w25q:W25Q U?
+U 1 1 5E861C02
+P 8800 5150
+F 0 "U?" H 8800 5625 50  0000 C CNN
+F 1 "W25Q" H 8800 5534 50  0000 C CNN
+F 2 "" H 8800 5250 50  0001 C CNN
+F 3 "" H 8800 5250 50  0001 C CNN
+	1    8800 5150
 	1    0    0    -1
 $EndComp
+Wire Wire Line
+	6700 3900 7100 3900
+Wire Wire Line
+	6700 4000 7100 4000
+Wire Wire Line
+	6700 4100 7100 4100
+Wire Wire Line
+	6700 4200 7100 4200
+Text Label 7100 3900 2    50   ~ 0
+iCE_MISO
+Text Label 7100 4000 2    50   ~ 0
+iCE_MOSI
+Text Label 7100 4100 2    50   ~ 0
+iCE_SCLK
+Text Label 7100 4200 2    50   ~ 0
+iCE_SS
+Entry Wire Line
+	2250 7450 2350 7550
+Wire Wire Line
+	2350 7550 2850 7550
+Text Label 2350 7550 0    50   ~ 0
+Om_SPI4
+Text Label 3100 7150 2    50   ~ 0
+iCE_MISO
+Text Label 3100 7350 2    50   ~ 0
+iCE_MOSI
+Text Label 3100 7250 2    50   ~ 0
+iCE_SCLK
+Text Label 3100 7450 2    50   ~ 0
+iCE_SS
+Wire Wire Line
+	2350 7150 3100 7150
+Wire Wire Line
+	2350 7250 3100 7250
+Wire Wire Line
+	2350 7350 3100 7350
+Wire Wire Line
+	2350 7450 3100 7450
+Wire Wire Line
+	9200 5000 9650 5000
+Wire Wire Line
+	9200 5100 9650 5100
+Wire Wire Line
+	9200 5200 9650 5200
+Wire Wire Line
+	9200 5400 9650 5400
+Text Label 9650 5000 2    50   ~ 0
+iCE_SCLK
+Text Label 9650 5100 2    50   ~ 0
+iCE_MISO
+Text Label 9650 5200 2    50   ~ 0
+iCE_MOSI
+Text Label 9650 4900 2    50   ~ 0
+iCE_SS
+$Comp
+L Device:R R?
+U 1 1 5E89BD86
+P 9650 5600
+F 0 "R?" H 9720 5646 50  0000 L CNN
+F 1 "R" H 9720 5555 50  0000 L CNN
+F 2 "" V 9580 5600 50  0001 C CNN
+F 3 "~" H 9650 5600 50  0001 C CNN
+	1    9650 5600
+	1    0    0    -1
+$EndComp
+$Comp
+L Device:R R?
+U 1 1 5E89D2A2
+P 9900 5600
+F 0 "R?" H 9970 5646 50  0000 L CNN
+F 1 "R" H 9970 5555 50  0000 L CNN
+F 2 "" V 9830 5600 50  0001 C CNN
+F 3 "~" H 9900 5600 50  0001 C CNN
+	1    9900 5600
+	1    0    0    -1
+$EndComp
+Wire Wire Line
+	9650 5400 9650 5450
+Wire Wire Line
+	9900 5300 9900 5450
+Wire Wire Line
+	9200 5300 9900 5300
+Wire Wire Line
+	9650 5750 9650 5900
+Wire Wire Line
+	9650 5900 9900 5900
+Wire Wire Line
+	9900 5900 9900 5750
+$Comp
+L Device:R R?
+U 1 1 5E89EE9F
+P 9900 4750
+F 0 "R?" H 9970 4796 50  0000 L CNN
+F 1 "R" H 9970 4705 50  0000 L CNN
+F 2 "" V 9830 4750 50  0001 C CNN
+F 3 "~" H 9900 4750 50  0001 C CNN
+	1    9900 4750
+	1    0    0    -1
+$EndComp
+Wire Wire Line
+	9200 4900 9900 4900
+Wire Bus Line
+	1200 6900 1200 7450
+Wire Bus Line
+	2250 6800 2250 7450
 $EndSCHEMATC

Commit message: Add files via upload
Parts:
- removed R?: R, symbol Device:R
- added C? (x2): 1u, symbol Device:C
- added C? (x11): 0.1u, symbol Device:C
- added C? (x3): 0.01u, symbol Device:C
- added C?: DNP, symbol Device:C
- added C? (x3): 10u, symbol Device:C
- added D?: CDBU0520, symbol Device:D_ALT
- added D?: GREEN, symbol Device:LED_ALT
- added D?: LED_RGB, symbol Device:LED_RGB
- added J? (x2): Conn_02x10_Odd_Even, symbol Connector_Generic:Conn_02x10_Odd_Even
- added Q?: S8550, Package_TO_SOT_THT:TO-92_Inline, symbol Transistor_BJT:S8550
- added R?: 100E, symbol Device:R
- added R? (x3): 2k2, symbol Device:R
- added R? (x2): 10K, symbol Device:R
- added R? (x2): 100, symbol Device:R
- added R? (x2): 10k, symbol Device:R
- added R? (x32): 33E, symbol Device:R
- added R?: 330, symbol Device:R
- added U?: HX711, symbol ADC:HX711
- added U?: ASFLMB-24.00MHZ-LC-T, symbol OSC:ASFLMB-24.00MHZ-LC-T
- added U?: SMS, symbol pulse:SMS
- R? (x2): value R -> 10k
Connections:
- net labels added: +1V2_FPGA, +3V3_FPGA, CLK_IN, COMM[3,0], CRESET_B, E+, E-, GND, IO1, IO10, IO11, IO12, IO13, IO14, IO15, IO16, IO17, IO18, IO19, IO2, IO20, IO21, IO22, IO23, IO24, IO25, IO3, IO4, IO5, IO6, IO7, IO8, IO9, RGB_B, RGB_G, RGB_R, S+, S-, SCK, SDA, SPIC_CS, SPIC_MISO, SPIC_MOSI, SPIC_SCLK
- net labels removed: COMM4, COMM[4,0]
- wire segments 25 -> 325
- no-connect marks 0 -> 1
Other:
- note added: "ALGUN REQUISITO ADICIONAL PARA EL OSCILADOR"
- note added: "CONDENSADOR DE DNP ENTRE VCC Y GND?"
- note added: "CONDENSADOR ES NECESARIO?"
- note added: "DEFINIR BOOT ONION"
- note added: "DEFINIR RELACION ENTRE R1 Y R2 O CAMBIAR EL ADC"
- note added: "PARA TODA SALIDA SE NECESITA?"
- note added: "QUE SIGNIFICA EL DNP Y CUAL DEBE SER EL DIODO"
- note added: "RESISTENCIA DE 33E PARA SDA Y SCK?"
- note added: "SE PUEDE PONER EL +5V DEL MCU?"
- moved on the sheet: R?, U?, U?A, U?B, U?C, U?D

Commit message: Add files via upload
Parts:
- removed C?: DNP, symbol Device:C
Other:
- note removed: "ALGUN REQUISITO ADICIONAL PARA EL OSCILADOR"
- note removed: "CONDENSADOR ES NECESARIO?"
Changed lines of the file:
@@
 Wire Wire Line
 	2700 1400 2700 1250
-Wire Wire Line
-	2700 1700 2700 1850
 $Comp
 L Device:D_ALT D?
@@
 $EndComp
 $Comp
-L Device:C C?
-U 1 1 5E9415E7
-P 3200 1550
-F 0 "C?" V 3150 1350 50  0000 L CNN
-F 1 "DNP" V 3150 1600 50  0000 L CNN
-F 2 "" H 3238 1400 50  0001 C CNN
-F 3 "~" H 3200 1550 50  0001 C CNN
-	1    3200 1550
-	1    0    0    -1
-$EndComp
-Wire Wire Line
-	3200 1400 3200 1250
-Wire Wire Line
-	3200 1700 3200 1850
-Wire Wire Line
-	3200 1850 2950 1850
-$Comp
 L power:GND #PWR?
 U 1 1 5E94F4B1
-P 2950 1900
-F 0 "#PWR?" H 2950 1650 50  0001 C CNN
-F 1 "GND" H 2955 1727 50  0000 C CNN
-F 2 "" H 2950 1900 50  0001 C CNN
-F 3 "" H 2950 1900 50  0001 C CNN
-	1    2950 1900
-	1    0    0    -1
-$EndComp
-Connection ~ 2950 1850
-Wire Wire Line
-	2950 1850 2700 1850
-Wire Wire Line
-	2950 1900 2950 1850
+P 2700 1900
+F 0 "#PWR?" H 2700 1650 50  0001 C CNN
+F 1 "GND" H 2705 1727 50  0000 C CNN
+F 2 "" H 2700 1900 50  0001 C CNN
+F 3 "" H 2700 1900 50  0001 C CNN
+	1    2700 1900
+	1    0    0    -1
+$EndComp
 Wire Wire Line
 	2700 1250 2800 1250
-Wire Wire Line
-	3100 1250 3200 1250
 Connection ~ 2700 1250
 Wire Wire Line
-	3200 1250 3750 1250
-Wire Wire Line
 	3750 1250 3750 2100
 Wire Wire Line
 	3750 2100 3850 2100
-Connection ~ 3200 1250
 $Comp
 L Device:R R?
@@
 Text Notes 13250 6250 2    50   ~ 0
 PARA TODA SALIDA SE NECESITA?
-Text Notes 12400 8050 2    50   ~ 0
-CONDENSADOR ES NECESARIO?
 $Comp
 L OSC:ASFLMB-24.00MHZ-LC-T U?
@@
 Wire Notes Line
 	3850 7750 7600 7750
+Wire Wire Line
+	3100 1250 3750 1250
+Wire Wire Line
+	2700 1700 2700 1900
 Wire Bus Line
 	4600 8250 4600 8800
 Wire Bus Line
 	6400 8250 6400 8900
-Text Notes 8100 7950 0    50   ~ 0
-ALGUN REQUISITO ADICIONAL PARA EL OSCILADOR
 $EndSCHEMATC

Commit message: Add files via upload
Other:
- note removed: "CONDENSADOR DE DNP ENTRE VCC Y GND?"
- note removed: "PARA TODA SALIDA SE NECESITA?"
- note removed: "RESISTENCIA DE 33E PARA SDA Y SCK?"
Changed lines of the file:
@@
 Text Notes 15000 2900 2    50   ~ 0
 DEFINIR RELACION ENTRE R1 Y R2 O CAMBIAR EL ADC
-Text Notes 12200 7600 2    50   ~ 0
-RESISTENCIA DE 33E PARA SDA Y SCK?
-Text Notes 14600 7600 2    50   ~ 0
-CONDENSADOR DE DNP ENTRE VCC Y GND?
-Text Notes 13250 6250 2    50   ~ 0
-PARA TODA SALIDA SE NECESITA?
 $Comp
 L OSC:ASFLMB-24.00MHZ-LC-T U?

Commit message: Add files via upload
Parts:
- J1, J2: renamed from J?; footprint (none) -> Connector_PinHeader_2.54mm:PinHeader_2x10_P2.54mm_Vertical
- gave numbers to parts that had none: 73

Commit message: Add files via upload
Parts:
- added R102, R103: 2K2, Resistor_SMD:R_0805_2012Metric_Pad1.15x1.40mm_HandSolder, symbol Device:R
- C1, C10, C11, C12, C13, C14, C15, C16, C17, C18, C19, C2, C5, C6, C7, C8: footprint (none) -> Capacitor_SMD:C_0805_2012Metric_Pad1.15x1.40mm_HandSolder
- C3, C4, C9: footprint (none) -> Capacitor_SMD:C_0603_1608Metric_Pad1.05x0.95mm_HandSolder
- D1, D2: footprint (none) -> LED_SMD:LED_0603_1608Metric_Pad1.05x0.95mm_HandSolder
- D3: footprint (none) -> LED_SMD:LED_RGB_Cree-PLCC-6_6x5mm_P2.1mm
- R1, R25, R26, R27, R3, R36, R4, R5, R6: footprint (none) -> Resistor_SMD:R_0603_1608Metric_Pad1.05x0.95mm_HandSolder
- R15, R16, R2: footprint (none) -> Resistor_SMD:R_0805_2012Metric_Pad1.15x1.40mm_HandSolder
- R37: value 330 -> 2K2; footprint (none) -> Resistor_SMD:R_0805_2012Metric_Pad1.15x1.40mm_HandSolder
Connections:
- net GND: now also R102.2, R103.2
- net at D3.1 (RK), R37.1: no longer D3.2 (GK), D3.3 (BK)
- new net: D3.2 (GK), R102.1
- new net: D3.3 (BK), R103.1

Commit message: Add files via upload
Parts:
- removed Q1: S8550, Package_TO_SOT_THT:TO-92_Inline, symbol Transistor_BJT:S8550
- added Q1: S8550, Package_TO_SOT_SMD:SOT-23, symbol Q_S8:S8550
- U2: footprint (none) -> AICE:ASFLMB
- U3: footprint (none) -> AICE:SMS_BUTTON
- U4: footprint (none) -> Package_SO:SOIC-8_5.23x5.23mm_P1.27mm
- U5: footprint (none) -> Package_SO:SOP-16_4.4x10.4mm_P1.27mm
Connections:
- net +3V3_FPGA: now also Q1.2 (E)
- net E+: now also Q1.3 (C)
- net at U5.2 (BASE): now also Q1.1 (B)
Changed lines of the file:
@@
 Text Label 4700 8900 0    50   ~ 0
 COMM3
-$Comp
-L w25q:W25Q U4
-U 1 1 5E861C02
-P 12200 5200
-F 0 "U4" H 12200 5675 50  0000 C CNN
-F 1 "W25Q" H 12200 5584 50  0000 C CNN
-F 2 "" H 12200 5300 50  0001 C CNN
-F 3 "" H 12200 5300 50  0001 C CNN
-	1    12200 5200
-	1    0    0    -1
-$EndComp
 Wire Wire Line
 	7700 6250 8100 6250
@@
 F 0 "U5" H 13550 2575 50  0000 C CNN
 F 1 "HX711" H 13550 2484 50  0000 C CNN
-F 2 "" H 13550 1800 50  0001 C CNN
+F 2 "Package_SO:SOP-16_4.4x10.4mm_P1.27mm" H 13550 1800 50  0001 C CNN
 F 3 "" H 13550 1800 50  0001 C CNN
 	1    13550 2000
@@
 	1    11500 3750
 	1    0    0    -1
-$EndComp
-$Comp
-L Transistor_BJT:S8550 Q1
-U 1 1 5E9AD2DF
-P 12000 1600
-F 0 "Q1" H 12191 1554 50  0000 L CNN
-F 1 "S8550" H 12191 1645 50  0000 L CNN
-F 2 "Package_TO_SOT_THT:TO-92_Inline" H 12200 1525 50  0001 L CIN
-F 3 "http://www.unisonic.com.tw/datasheet/S8550.pdf" H 12000 1600 50  0001 L CNN
-	1    12000 1600
-	-1   0    0    1
 $EndComp
 $Comp
@@
 F 0 "U3" H 11550 9225 50  0000 C CNN
 F 1 "SMS" H 11550 9134 50  0000 C CNN
-F 2 "" H 11950 9150 50  0001 C CNN
+F 2 "AICE:SMS_BUTTON" H 11950 9150 50  0001 C CNN
 F 3 "" H 11950 9150 50  0001 C CNN
 	1    11550 8950
@@
 F 0 "U2" H 9000 8975 50  0000 C CNN
 F 1 "ASFLMB-24.00MHZ-LC-T" H 9000 8884 50  0000 C CNN
-F 2 "" H 9000 9000 50  0001 C CNN
+F 2 "AICE:ASFLMB" H 9000 9000 50  0001 C CNN
 F 3 "" H 9000 9000 50  0001 C CNN
 	1    9000 8650
@@
 	1    0    0    -1
 $EndComp
+$Comp
+L w25q:W25Q U4
+U 1 1 5E861C02
+P 12200 5200
+F 0 "U4" H 12200 5675 50  0000 C CNN
+F 1 "W25Q" H 12200 5584 50  0000 C CNN
+F 2 "Package_SO:SOIC-8_5.23x5.23mm_P1.27mm" H 12200 5300 50  0001 C CNN
+F 3 "" H 12200 5300 50  0001 C CNN
+	1    12200 5200
+	1    0    0    -1
+$EndComp
 Wire Bus Line
 	4600 8250 4600 8800
 Wire Bus Line
 	6400 8250 6400 8900
+$Comp
+L Q_S8:S8550 Q1
+U 1 1 5EB3D4A0
+P 12000 1600
+F 0 "Q1" H 12191 1554 50  0000 L CNN
+F 1 "S8550" H 12191 1645 50  0000 L CNN
+F 2 "Package_TO_SOT_SMD:SOT-23" H 12300 1700 50  0001 C CNN
+F 3 "" H 12300 1700 50  0001 C CNN
+	1    12000 1600
+	-1   0    0    1
+$EndComp
 $EndSCHEMATC

Commit message: Add files via upload
Parts:
- removed R10, R11, R12, R13, R14, R17, R18, R19, R20, R21, R22, R23, R24, R28, R29, R30, R31, R32, R33, R34, R35, R38, R39, R40, R41, R42, R43, R44, R45, R7, R8, R9: 33E, symbol Device:R
- C1, C10, C11, C12, C13, C14, C15, C16, C17, C18, C19, C2, C5, C6, C7, C8: footprint Capacitor_SMD:C_0805_2012Metric_Pad1.15x1.40mm_HandSolder -> Capacitor_SMD:C_0603_1608Metric_Pad1.05x0.95mm_HandSolder
- R102, R103, R15, R16, R2, R37: footprint Resistor_SMD:R_0805_2012Metric_Pad1.15x1.40mm_HandSolder -> Resistor_SMD:R_0603_1608Metric_Pad1.05x0.95mm_HandSolder
Connections:
- net E+: now also J2.16 (Pin_16)
- net IO1: now also J1.5 (Pin_5)
- net IO10: now also J1.14 (Pin_14)
- net IO11: now also J1.15 (Pin_15)
- net IO12: now also J1.16 (Pin_16)
- net IO13: now also J1.17 (Pin_17)
- net IO14: now also J1.18 (Pin_18)
- net IO15: now also J2.5 (Pin_5)
- net IO16: now also J2.6 (Pin_6)
- net IO17: now also J2.7 (Pin_7)
- net IO18: now also J2.8 (Pin_8)
- net IO19: now also J2.9 (Pin_9)
- net IO2: now also J1.6 (Pin_6)
- net IO20: now also J2.10 (Pin_10)
- net IO21: now also J2.11 (Pin_11)
- net IO22: now also J2.12 (Pin_12)
- net IO23: now also J2.13 (Pin_13)
- net IO24: now also J2.14 (Pin_14)
- net IO25: now also J2.15 (Pin_15)
- net IO3: now also J1.7 (Pin_7)
- net IO4: now also J1.8 (Pin_8)
- net IO5: now also J1.9 (Pin_9)
- net IO6: now also J1.10 (Pin_10)
- net IO7: now also J1.11 (Pin_11)
- net IO8: now also J1.12 (Pin_12)
- net IO9: now also J1.13 (Pin_13)
- net S+: now also J2.17 (Pin_17)
- net S-: now also J2.18 (Pin_18)
- net SCK: now also J1.20 (Pin_20), J2.19 (Pin_19)
- net SDA: now also J1.19 (Pin_19), J2.20 (Pin_20)
- net Om_SPI0 renamed OmSPI0
- net Om_SPI1 renamed OmSPI1
- net Om_SPI2 renamed OmSPI2
- net Om_SPI3 renamed OmSPI3
