File: AICE/iCE40.sch (KiCad schematic (older format))
At the start: 45 parts, among them J1 Conn_02x10_Odd_Even, J2 Conn_02x10_Odd_Even, Q1 S8550, U1 ICE40UP5K-SG48ITR, U2 ASFLMB-24.00MHZ-LC-T, U3 SMS, U4 W25Q, U5 HX711

Commit message: Add files via upload
Connections:
- net COMM0: now also U1.21 (IOB_23b); no longer U1.36 (IOT_48b)
- net COMM1: now also U1.20 (IOB_25b_G3); no longer U1.43 (IOT_49a)
- net COMM2: now also U1.19 (IOB_29b); no longer U1.38 (IOT_50b)
- net COMM3: now also U1.18 (IOB_31b); no longer U1.42 (IOT_51a)
- net E+: now also J2.10 (Pin_10); no longer J2.16 (Pin_16)
- net IO1: now also U1.13 (IOB_24a); no longer U1.46 (IOB_0a)
- net IO10: now also U1.48 (IOB_4a); no longer U1.9 (IOB_16a)
- net IO11: now also U1.46 (IOB_0a); no longer U1.10 (IOB_18a)
- net IO12: now also U1.47 (IOB_2a); no longer U1.11 (IOB_20a)
- net IO13: now also U1.44 (IOB_3b_G6); no longer U1.12 (IOB_22b)
- net IO14: now also U1.45 (IOB_5b); no longer U1.21 (IOB_23b)
- net IO15: now also J1.19 (Pin_19), U1.42 (IOT_51a); no longer J2.5 (Pin_5), U1.13 (IOB_24a)
- net IO16: now also J1.20 (Pin_20), U1.43 (IOT_49a); no longer J2.6 (Pin_6), U1.20 (IOB_25b_G3)
- net IO17: now also J2.11 (Pin_11), U1.31 (IOT_42b); no longer J2.7 (Pin_7), U1.19 (IOB_29b)
- net IO18: now also J2.14 (Pin_14), U1.32 (IOT_43a); no longer J2.8 (Pin_8), U1.18 (IOB_31b)
- net IO19: now also J2.13 (Pin_13), U1.34 (IOT_44b); no longer J2.9 (Pin_9), U1.25 (IOT_36b)
- net IO2: now also U1.12 (IOB_22b); no longer U1.47 (IOB_2a)
- net IO20: now also J2.16 (Pin_16), U1.36 (IOT_48b); no longer J2.10 (Pin_10), U1.23 (IOT_37a)
- net IO21: now also J2.15 (Pin_15), U1.37 (IOT_45a_G1); no longer J2.11 (Pin_11), U1.27 (IOT_38b)
- net IO22: now also J2.18 (Pin_18), U1.38 (IOT_50b); no longer J2.12 (Pin_12), U1.26 (IOT_39a)
- net IO23: now also J2.17 (Pin_17), U1.39 (RGB0); no longer J2.13 (Pin_13), U1.28 (IOT_41a)
- net IO24: now also J2.20 (Pin_20), U1.40 (RGB1); no longer J2.14 (Pin_14), U1.31 (IOT_42b)
- net IO25: now also J2.19 (Pin_19), U1.41 (RGB2); no longer J2.15 (Pin_15), U1.32 (IOT_43a)
- net IO3: now also U1.11 (IOB_20a); no longer U1.44 (IOB_3b_G6)
- net IO4: now also U1.10 (IOB_18a); no longer U1.48 (IOB_4a)
- net IO5: now also U1.9 (IOB_16a); no longer U1.45 (IOB_5b)
- net IO6: now also U1.6 (IOB_13b); no longer U1.2 (IOB_6a)
- net IO9: now also U1.2 (IOB_6a); no longer U1.6 (IOB_13b)
- net RGB_B: now also U1.26 (IOT_39a); no longer U1.41 (RGB2)
- net RGB_G: now also U1.25 (IOT_36b); no longer U1.40 (RGB1)
- net RGB_R: now also U1.23 (IOT_37a); no longer U1.39 (RGB0)
- net S+: now also J2.9 (Pin_9); no longer J2.17 (Pin_17)
- net S-: now also J2.12 (Pin_12); no longer J2.18 (Pin_18)
- net SCK: now also J2.7 (Pin_7), J2.8 (Pin_8), U1.28 (IOT_41a); no longer J1.20 (Pin_20), J2.19 (Pin_19), U1.34 (IOT_44b)
- net SDA: now also J2.5 (Pin_5), J2.6 (Pin_6), U1.27 (IOT_38b); no longer J1.19 (Pin_19), J2.20 (Pin_20), U1.37 (IOT_45a_G1)
Changed lines of the file:
@@
 	5950 2800 5650 2800
 Text Label 5650 2800 0    50   ~ 0
-IO1
+IO11
 Wire Wire Line
 	5950 2900 5650 2900
 Text Label 5650 2900 0    50   ~ 0
-IO2
+IO12
 Wire Wire Line
 	5950 3000 5650 3000
 Text Label 5650 3000 0    50   ~ 0
-IO3
+IO13
 Wire Wire Line
 	5950 3100 5650 3100
 Text Label 5650 3100 0    50   ~ 0
-IO4
+IO10
 Wire Wire Line
 	5950 3200 5650 3200
 Text Label 5650 3200 0    50   ~ 0
-IO5
+IO14
 Wire Wire Line
 	5950 3300 5650 3300
 Text Label 5650 3300 0    50   ~ 0
-IO6
+IO9
 Wire Wire Line
 	5950 3400 5650 3400
@@
 IO8
 Wire Wire Line
-	4550 4950 4250 4950
-Text Label 4250 4950 0    50   ~ 0
-IO19
-Wire Wire Line
-	4550 5050 4250 5050
-Text Label 4250 5050 0    50   ~ 0
-IO20
-Wire Wire Line
 	4550 5150 4250 5150
 Text Label 4250 5150 0    50   ~ 0
-IO21
-Wire Wire Line
-	4550 5250 4250 5250
-Text Label 4250 5250 0    50   ~ 0
-IO22
+SDA
 Wire Wire Line
 	4550 5350 4250 5350
 Text Label 4250 5350 0    50   ~ 0
-IO23
+SCK
 Wire Wire Line
 	4550 5450 4250 5450
 Text Label 4250 5450 0    50   ~ 0
-IO24
+IO17
 Wire Wire Line
 	4550 5550 4250 5550
 Text Label 4250 5550 0    50   ~ 0
-IO25
+IO18
 Wire Wire Line
 	4550 5850 4250 5850
@@
 	4550 5650 4250 5650
 Text Label 4250 5650 0    50   ~ 0
-SCK
+IO19
 Wire Wire Line
 	4550 5750 4250 5750
 Text Label 4250 5750 0    50   ~ 0
-SDA
+IO21
 Wire Wire Line
 	7700 5250 8000 5250
 Text Label 8000 5250 2    50   ~ 0
-IO9
+IO6
 Wire Wire Line
 	7700 5350 8000 5350
 Text Label 8000 5350 2    50   ~ 0
-IO10
+IO5
 Wire Wire Line
 	7700 5450 8000 5450
 Text Label 8000 5450 2    50   ~ 0
-IO11
+IO4
 Wire Wire Line
 	7700 5550 8000 5550
 Text Label 8000 5550 2    50   ~ 0
-IO12
+IO3
 Wire Wire Line
 	7700 5650 8000 5650
 Text Label 8000 5650 2    50   ~ 0
-IO13
-Wire Wire Line
-	7700 5750 8000 5750
-Text Label 8000 5750 2    50   ~ 0
-IO14
-Wire Wire Line
-	7700 5850 8000 5850
-Text Label 8000 5850 2    50   ~ 0
-IO15
-Wire Wire Line
-	7700 5950 8000 5950
-Text Label 8000 5950 2    50   ~ 0
-IO16
-Wire Wire Line
-	7700 6050 8000 6050
-Text Label 8000 6050 2    50   ~ 0
-IO17
-Wire Wire Line
-	7700 6150 8000 6150
-Text Label 8000 6150 2    50   ~ 0
-IO18
+IO2
 $Comp
 L power:GND #PWR016
@@
 Text Label 12200 7250 2    50   ~ 0
 IO14
-Text Label 11000 7350 0    50   ~ 0
+Text Label 13200 6650 0    50   ~ 0
 SDA
-Text Label 12200 7350 2    50   ~ 0
+Text Label 14400 6750 2    50   ~ 0
 SCK
 $Comp
@@
 Wire Wire Line
 	13450 6500 13450 6550
-Text Label 14400 6650 2    50   ~ 0
+Text Label 12200 7350 2    50   ~ 0
 IO16
-Text Label 14400 6750 2    50   ~ 0
+Text Label 14400 7050 2    50   ~ 0
 IO18
+Text Label 14400 7150 2    50   ~ 0
+IO20
+Text Label 14400 7250 2    50   ~ 0
+IO22
+Text Label 14400 7350 2    50   ~ 0
+IO24
+Wire Notes Line
+	10400 6100 10400 7700
+Wire Notes Line
+	10400 7700 15050 7700
+Wire Notes Line
+	15050 7700 15050 6100
+Wire Notes Line
+	15050 6100 10400 6100
 Text Label 14400 6850 2    50   ~ 0
-IO20
+E+
 Text Label 14400 6950 2    50   ~ 0
-IO22
-Text Label 14400 7050 2    50   ~ 0
-IO24
-Text Label 14400 7350 2    50   ~ 0
-SDA
-Wire Notes Line
-	10400 6100 10400 7700
-Wire Notes Line
-	10400 7700 15050 7700
-Wire Notes Line
-	15050 7700 15050 6100
-Wire Notes Line
-	15050 6100 10400 6100
-Text Label 14400 7150 2    50   ~ 0
-E+
-Text Label 14400 7250 2    50   ~ 0
 S-
 Text Label 11000 7250 0    50   ~ 0
@@
 	4550 6350 4250 6350
 Text Label 4250 6350 0    50   ~ 0
-RGB_R
+IO23
 Wire Wire Line
 	4550 6450 4250 6450
 Text Label 4250 6450 0    50   ~ 0
-RGB_G
+IO24
 Wire Wire Line
 	4550 6550 4250 6550
 Text Label 4250 6550 0    50   ~ 0
-RGB_B
+IO25
 Wire Wire Line
 	7700 4950 8100 4950
@@
 	11000 7250 11350 7250
 Wire Wire Line
+	13200 6650 13550 6650
+Wire Wire Line
+	11850 6650 12200 6650
+Wire Wire Line
+	11850 6750 12200 6750
+Wire Wire Line
+	11850 6850 12200 6850
+Wire Wire Line
+	11850 6950 12200 6950
+Wire Wire Line
+	11850 7050 12200 7050
+Wire Wire Line
+	11850 7150 12200 7150
+Wire Wire Line
+	11850 7250 12200 7250
+Wire Wire Line
+	14050 6750 14400 6750
+Text Label 11000 7350 0    50   ~ 0
+IO15
+Text Label 13200 6850 0    50   ~ 0
+S+
+Text Label 13200 6750 0    50   ~ 0
+SCK
+Text Label 13200 7350 0    50   ~ 0
+IO25
+Text Label 13200 7250 0    50   ~ 0
+IO23
+Text Label 13200 7150 0    50   ~ 0
+IO21
+Text Label 13200 7050 0    50   ~ 0
+IO19
+Text Label 13200 6950 0    50   ~ 0
+IO17
+Wire Wire Line
 	11000 7350 11350 7350
 Wire Wire Line
-	11850 6650 12200 6650
-Wire Wire Line
-	11850 6750 12200 6750
-Wire Wire Line
-	11850 6850 12200 6850
-Wire Wire Line
-	11850 6950 12200 6950
-Wire Wire Line
-	11850 7050 12200 7050
-Wire Wire Line
-	11850 7150 12200 7150
-Wire Wire Line
-	11850 7250 12200 7250
+	13200 6950 13550 6950
+Wire Wire Line
+	13200 7050 13550 7050
+Wire Wire Line
+	13200 7150 13550 7150
+Wire Wire Line
+	13200 7250 13550 7250
+Wire Wire Line
+	13200 7350 13550 7350
+Wire Wire Line
+	13200 6850 13550 6850
+Wire Wire Line
+	13200 6750 13550 6750
 Wire Wire Line
 	11850 7350 12200 7350
-Text Label 13200 6650 0    50   ~ 0
+Wire Wire Line
+	14050 7050 14400 7050
+Wire Wire Line
+	14050 7150 14400 7150
+Wire Wire Line
+	14050 7250 14400 7250
+Wire Wire Line
+	14050 7350 14400 7350
+Wire Wire Line
+	14050 6850 14400 6850
+Wire Wire Line
+	14050 6950 14400 6950
+Text Label 4100 5950 0    50   ~ 0
+IO20
+Text Label 4100 6050 0    50   ~ 0
+IO16
+Text Label 4100 6150 0    50   ~ 0
+IO22
+Text Label 4100 6250 0    50   ~ 0
 IO15
-Text Label 13200 7250 0    50   ~ 0
-S+
-Text Label 13200 7350 0    50   ~ 0
-SCK
-Text Label 13200 7150 0    50   ~ 0
-IO25
-Text Label 13200 7050 0    50   ~ 0
-IO23
-Text Label 13200 6950 0    50   ~ 0
-IO21
-Text Label 13200 6850 0    50   ~ 0
-IO19
-Text Label 13200 6750 0    50   ~ 0
-IO17
-Wire Wire Line
-	13200 6650 13550 6650
-Wire Wire Line
-	13200 6750 13550 6750
-Wire Wire Line
-	13200 6850 13550 6850
-Wire Wire Line
-	13200 6950 13550 6950
-Wire Wire Line
-	13200 7050 13550 7050
-Wire Wire Line
-	13200 7150 13550 7150
-Wire Wire Line
-	13200 7250 13550 7250
-Wire Wire Line
-	13200 7350 13550 7350
-Wire Wire Line
-	14050 6650 14400 6650
-Wire Wire Line
-	14050 6750 14400 6750
-Wire Wire Line
-	14050 6850 14400 6850
-Wire Wire Line
-	14050 6950 14400 6950
-Wire Wire Line
-	14050 7050 14400 7050
-Wire Wire Line
-	14050 7350 14400 7350
-Wire Wire Line
-	14050 7150 14400 7150
-Wire Wire Line
-	14050 7250 14400 7250
-Text Label 4100 5950 0    50   ~ 0
-SPIC_MISO
-Text Label 4100 6050 0    50   ~ 0
-SPIC_SCLK
-Text Label 4100 6150 0    50   ~ 0
-SPIC_MOSI
-Text Label 4100 6250 0    50   ~ 0
-SPIC_CS
 Wire Wire Line
 	4550 5950 4100 5950
@@
 	0    -1   -1   0
 $EndComp
-Wire Bus Line
-	6400 8250 6400 8900
-Wire Bus Line
-	4600 8250 4600 8800
 $Comp
 L Device:LED_ALT D2
@@
 	0    -1   -1   0
 $EndComp
+Wire Wire Line
+	7700 5850 8000 5850
+Wire Wire Line
+	7700 5750 8450 5750
+Text Label 8450 5750 2    50   ~ 0
+SPIC_MISO
+Wire Wire Line
+	7700 5950 8450 5950
+Wire Wire Line
+	7700 6050 8450 6050
+Wire Wire Line
+	7700 6150 8450 6150
+Text Label 8450 6150 2    50   ~ 0
+SPIC_CS
+Text Label 8450 6050 2    50   ~ 0
+SPIC_MOSI
+Text Label 8450 5950 2    50   ~ 0
+SPIC_SCLK
+Text Label 8000 5850 2    50   ~ 0
+IO1
+Wire Wire Line
+	14050 6650 14400 6650
+Text Label 14400 6650 2    50   ~ 0
+SDA
+Text Label 4250 5050 0    50   ~ 0
+RGB_R
+Text Label 4250 4950 0    50   ~ 0
+RGB_G
+Text Label 4250 5250 0    50   ~ 0
+RGB_B
+Wire Wire Line
+	4250 5250 4550 5250
+Wire Wire Line
+	4250 4950 4550 4950
+Wire Wire Line
+	4250 5050 4550 5050
+Wire Bus Line
+	4600 8250 4600 8800
+Wire Bus Line
+	6400 8250 6400 8900
 $EndSCHEMATC

Commit message: Add files via upload
Parts:
- C1, C10, C11, C12, C13, C14, C15, C16, C17, C18, C19, C2, C3, C4, C5, C6, C7, C8, C9: footprint Capacitor_SMD:C_0603_1608Metric_Pad1.05x0.95mm_HandSolder -> Capacitor_SMD:C_0603_1608Metric
- D1, D2: footprint LED_SMD:LED_0603_1608Metric_Pad1.05x0.95mm_HandSolder -> LED_SMD:LED_0603_1608Metric
- R1, R102, R103, R15, R16, R2, R25, R26, R27, R3, R36, R37, R4, R5, R6: footprint Resistor_SMD:R_0603_1608Metric_Pad1.05x0.95mm_HandSolder -> Resistor_SMD:R_0603_1608Metric
Connections:
- net E+: now also J2.6 (Pin_6); no longer J2.10 (Pin_10)
- net IO11: now also U1.47 (IOB_2a); no longer U1.46 (IOB_0a)
- net IO12: now also U1.46 (IOB_0a); no longer U1.47 (IOB_2a)
- net IO13: now also U1.45 (IOB_5b); no longer U1.44 (IOB_3b_G6)
- net IO14: now also U1.44 (IOB_3b_G6); no longer U1.45 (IOB_5b)
- net IO15: now also U1.43 (IOT_49a); no longer U1.42 (IOT_51a)
- net IO16: now also U1.42 (IOT_51a); no longer U1.43 (IOT_49a)
- net S+: now also J2.5 (Pin_5); no longer J2.9 (Pin_9)
- net S-: now also J2.8 (Pin_8); no longer J2.12 (Pin_12)
- net SCK: now also J2.12 (Pin_12), J2.9 (Pin_9); no longer J2.7 (Pin_7), J2.8 (Pin_8)
- net SDA: now also J2.10 (Pin_10), J2.7 (Pin_7); no longer J2.5 (Pin_5), J2.6 (Pin_6)

Commit message: Add files via upload
Connections:
- net SCK: now also J2.10 (Pin_10), J2.7 (Pin_7), U1.27 (IOT_38b); no longer J2.12 (Pin_12), J2.9 (Pin_9), U1.28 (IOT_41a)
- net SDA: now also J2.12 (Pin_12), J2.9 (Pin_9), U1.28 (IOT_41a); no longer J2.10 (Pin_10), J2.7 (Pin_7), U1.27 (IOT_38b)
Changed lines of the file:
@@
 IO8
+Wire Wire Line
+	4550 5350 4250 5350
+Text Label 4250 5350 0    50   ~ 0
+SDA
 Wire Wire Line
 	4550 5150 4250 5150
 Text Label 4250 5150 0    50   ~ 0
-SDA
-Wire Wire Line
-	4550 5350 4250 5350
-Text Label 4250 5350 0    50   ~ 0
 SCK
 Wire Wire Line
@@
 Text Label 12200 7250 2    50   ~ 0
 IO14
-Text Label 13200 6750 0    50   ~ 0
+Text Label 13200 6850 0    50   ~ 0
 SDA
-Text Label 14400 6950 2    50   ~ 0
+Text Label 14400 6850 2    50   ~ 0
 SCK
 $Comp
@@
 	11000 7250 11350 7250
 Wire Wire Line
-	13200 6750 13550 6750
+	13200 6850 13550 6850
 Wire Wire Line
 	11850 6650 12200 6650
@@
 	11850 7250 12200 7250
 Wire Wire Line
-	14050 6950 14400 6950
+	14050 6850 14400 6850
 Text Label 11000 7350 0    50   ~ 0
 IO15
 Text Label 13200 6650 0    50   ~ 0
 S+
-Text Label 13200 6850 0    50   ~ 0
+Text Label 13200 6750 0    50   ~ 0
 SCK
 Text Label 13200 7350 0    50   ~ 0
@@
 	13200 6650 13550 6650
 Wire Wire Line
-	13200 6850 13550 6850
+	13200 6750 13550 6750
 Wire Wire Line
 	11850 7350 12200 7350
@@
 IO1
 Wire Wire Line
-	14050 6850 14400 6850
-Text Label 14400 6850 2    50   ~ 0
+	14050 6950 14400 6950
+Text Label 14400 6950 2    50   ~ 0
 SDA
 Text Label 4250 5050 0    50   ~ 0
