File: AICE/sipeedm1w.sch (KiCad schematic (older format))
At the start: 1 part

Commit message: Add files via upload
Parts:
- added C? (x4): 0.1u, symbol Device:C
Connections:
- net GND: now reaches U?.0 (GND)
- net GND: now also U?.49 (GND), U?.50 (GND), U?.72 (GND), C?.1, C?.1, C?.1, C?.1
- net +5V_MCU: now reaches U?.51 (5V)
- net +5V_MCU: now also U?.52 (5V), C?.2, C?.2
- net +1V8_MCU: now reaches U?.53 (1V8)
- net +1V8_MCU: now also C?.2
- net +3V3_MCU: now reaches U?.54 (3V3)
- net +3V3_MCU: now also C?.2
Changed lines of the file:
@@
 $Descr A4 11693 8268
 encoding utf-8
-Sheet 4 4
+Sheet 4 5
 Title ""
 Date ""
@@
 	1300 6700 1100 6700
 Text HLabel 1100 6700 0    50   BiDi ~ 0
-COMM[4,0]
+COMM[3,0]
 Text Label 4300 2950 0    50   ~ 0
 TCK
@@
 Text HLabel 4300 3950 0    50   Output ~ 0
 TX_M1
+$Comp
+L power:GND #PWR?
+U 1 1 5EB07062
+P 6950 5350
+F 0 "#PWR?" H 6950 5100 50  0001 C CNN
+F 1 "GND" H 6955 5177 50  0000 C CNN
+F 2 "" H 6950 5350 50  0001 C CNN
+F 3 "" H 6950 5350 50  0001 C CNN
+	1    6950 5350
+	1    0    0    -1
+$EndComp
+$Comp
+L power:GND #PWR?
+U 1 1 5EB07767
+P 4850 5350
+F 0 "#PWR?" H 4850 5100 50  0001 C CNN
+F 1 "GND" H 4855 5177 50  0000 C CNN
+F 2 "" H 4850 5350 50  0001 C CNN
+F 3 "" H 4850 5350 50  0001 C CNN
+	1    4850 5350
+	1    0    0    -1
+$EndComp
+$Comp
+L power:GND #PWR?
+U 1 1 5EB07C18
+P 6950 2300
+F 0 "#PWR?" H 6950 2050 50  0001 C CNN
+F 1 "GND" H 6955 2127 50  0000 C CNN
+F 2 "" H 6950 2300 50  0001 C CNN
+F 3 "" H 6950 2300 50  0001 C CNN
+	1    6950 2300
+	-1   0    0    1
+$EndComp
+$Comp
+L power:GND #PWR?
+U 1 1 5EB09351
+P 7600 3450
+F 0 "#PWR?" H 7600 3200 50  0001 C CNN
+F 1 "GND" V 7605 3322 50  0000 R CNN
+F 2 "" H 7600 3450 50  0001 C CNN
+F 3 "" H 7600 3450 50  0001 C CNN
+	1    7600 3450
+	0    -1   -1   0
+$EndComp
+Wire Wire Line
+	7250 3450 7350 3450
+Wire Wire Line
+	7250 3350 7350 3350
+Wire Wire Line
+	7350 3350 7350 3450
+Connection ~ 7350 3450
+Wire Wire Line
+	7350 3450 7600 3450
+Wire Wire Line
+	6950 5350 6950 5150
+Wire Wire Line
+	4850 5150 4850 5350
+Wire Wire Line
+	6950 2450 6950 2300
+$Comp
+L Device:C C?
+U 1 1 5EB10615
+P 10150 1450
+AR Path="/5E829221/5EB10615" Ref="C?"  Part="1"
+AR Path="/5E828FD1/5EB10615" Ref="C?"  Part="1"
+F 0 "C?" V 10100 1250 50  0000 L CNN
+F 1 "0.1u" V 10100 1500 50  0000 L CNN
+F 2 "" H 10188 1300 50  0001 C CNN
+F 3 "~" H 10150 1450 50  0001 C CNN
+	1    10150 1450
+	-1   0    0    1
+$EndComp
+$Comp
+L Device:C C?
+U 1 1 5EB1C0E1
+P 10400 1450
+AR Path="/5E829221/5EB1C0E1" Ref="C?"  Part="1"
+AR Path="/5E828FD1/5EB1C0E1" Ref="C?"  Part="1"
+F 0 "C?" V 10350 1250 50  0000 L CNN
+F 1 "0.1u" V 10350 1500 50  0000 L CNN
+F 2 "" H 10438 1300 50  0001 C CNN
+F 3 "~" H 10400 1450 50  0001 C CNN
+	1    10400 1450
+	-1   0    0    1
+$EndComp
+Wire Wire Line
+	10400 1200 10400 1300
+Wire Wire Line
+	10150 1300 10150 1200
+Wire Wire Line
+	10150 1600 10150 1750
+Wire Wire Line
+	10150 1750 10300 1750
+Wire Wire Line
+	10400 1750 10400 1600
+$Comp
+L power:GND #PWR?
+U 1 1 5EB22A39
+P 10300 1900
+F 0 "#PWR?" H 10300 1650 50  0001 C CNN
+F 1 "GND" H 10305 1727 50  0000 C CNN
+F 2 "" H 10300 1900 50  0001 C CNN
+F 3 "" H 10300 1900 50  0001 C CNN
+	1    10300 1900
+	1    0    0    -1
+$EndComp
+Wire Wire Line
+	10300 1900 10300 1750
+Connection ~ 10300 1750
+Wire Wire Line
+	10300 1750 10400 1750
+Text GLabel 10700 1200 2    50   Input ~ 0
++5V_MCU
+Wire Wire Line
+	7250 3150 7550 3150
+Wire Wire Line
+	7550 3150 7550 3250
+Wire Wire Line
+	7550 3250 7250 3250
+Text Label 7500 3150 2    50   ~ 0
++5V
+Text Label 7550 3050 2    50   ~ 0
++1V8
+Text Label 7550 2950 2    50   ~ 0
++3V3
+Wire Wire Line
+	7250 2950 7550 2950
+Wire Wire Line
+	7250 3050 7550 3050
+Connection ~ 10150 1200
+Wire Wire Line
+	10150 1200 10400 1200
+Connection ~ 10400 1200
+Wire Wire Line
+	10400 1200 10700 1200
+Text Label 9900 1200 0    50   ~ 0
++5V
+Wire Wire Line
+	9900 1200 10150 1200
+$Comp
+L Device:C C?
+U 1 1 5EB44339
+P 10300 2450
+AR Path="/5E829221/5EB44339" Ref="C?"  Part="1"
+AR Path="/5E828FD1/5EB44339" Ref="C?"  Part="1"
+F 0 "C?" V 10250 2250 50  0000 L CNN
+F 1 "0.1u" V 10250 2500 50  0000 L CNN
+F 2 "" H 10338 2300 50  0001 C CNN
+F 3 "~" H 10300 2450 50  0001 C CNN
+	1    10300 2450
+	-1   0    0    1
+$EndComp
+Wire Wire Line
+	10300 2300 10300 2200
+Wire Wire Line
+	10300 2600 10300 2750
+Text GLabel 10650 2200 2    50   Input ~ 0
++3V3_MCU
+Wire Wire Line
+	10300 2200 9900 2200
+Text Label 9900 2200 0    50   ~ 0
++3V3
+$Comp
+L power:GND #PWR?
+U 1 1 5EB4C66B
+P 10300 2750
+F 0 "#PWR?" H 10300 2500 50  0001 C CNN
+F 1 "GND" H 10305 2577 50  0000 C CNN
+F 2 "" H 10300 2750 50  0001 C CNN
+F 3 "" H 10300 2750 50  0001 C CNN
+	1    10300 2750
+	1    0    0    -1
+$EndComp
+Wire Wire Line
+	10300 2200 10650 2200
+Connection ~ 10300 2200
+$Comp
+L Device:C C?
+U 1 1 5EB53904
+P 10300 3250
+AR Path="/5E829221/5EB53904" Ref="C?"  Part="1"
+AR Path="/5E828FD1/5EB53904" Ref="C?"  Part="1"
+F 0 "C?" V 10250 3050 50  0000 L CNN
+F 1 "0.1u" V 10250 3300 50  0000 L CNN
+F 2 "" H 10338 3100 50  0001 C CNN
+F 3 "~" H 10300 3250 50  0001 C CNN
+	1    10300 3250
+	-1   0    0    1
+$EndComp
+Wire Wire Line
+	10300 3100 10300 3000
+Wire Wire Line
+	10300 3400 10300 3550
+Text GLabel 10650 3000 2    50   Input ~ 0
++1V8_MCU
+Wire Wire Line
+	10300 3000 9900 3000
+Text Label 9900 3000 0    50   ~ 0
++1V8
+$Comp
+L power:GND #PWR?
+U 1 1 5EB5390F
+P 10300 3550
+F 0 "#PWR?" H 10300 3300 50  0001 C CNN
+F 1 "GND" H 10305 3377 50  0000 C CNN
+F 2 "" H 10300 3550 50  0001 C CNN
+F 3 "" H 10300 3550 50  0001 C CNN
+	1    10300 3550
+	1    0    0    -1
+$EndComp
+Wire Wire Line
+	10300 3000 10650 3000
+Connection ~ 10300 3000
+$Comp
+L power:GND #PWR?
+U 1 1 5EB59EFD
+P 5050 2300
+F 0 "#PWR?" H 5050 2050 50  0001 C CNN
+F 1 "GND" H 5055 2127 50  0000 C CNN
+F 2 "" H 5050 2300 50  0001 C CNN
+F 3 "" H 5050 2300 50  0001 C CNN
+	1    5050 2300
+	-1   0    0    1
+$EndComp
+Wire Wire Line
+	5050 2450 5050 2300
 Wire Bus Line
 	1300 6700 1300 7350

Commit message: Add files via upload
Parts:
- removed U?: M1&M1W, symbol M1&M1w:M1&M1W
- added U?: M1&M1W, symbol M1&M1w:M1&M1W
Connections:
- net +1V8_MCU: now also U?.53 (1V8)
- net +3V3_MCU: now also U?.54 (3V3)
- net +5V_MCU: now also U?.51 (5V), U?.52 (5V)
- net COMM0: now also U?.27 (IO26)
- net COMM1: now also U?.28 (IO27)
- net COMM2: now also U?.29 (IO28)
- net COMM3: now also U?.30 (IO29)
- net GND: now also U?.0 (GND), U?.49 (GND), U?.50 (GND), U?.72 (GND)
- net JTAG0: now also U?.3 (IO2)
- net JTAG1: now also U?.1 (IO0)
- net JTAG2: now also U?.2 (IO1)
- net JTAG3: now also U?.4 (IO3)
- net RX_M1: now also U?.10 (IO9)
- net SPIO_CS1: now also U?.26 (IO25)
- net TX_M1: now also U?.11 (IO10)
Changed lines of the file:
@@
 Comment4 ""
 $EndDescr
-$Comp
-L M1&M1w:M1&M1W U?
-U 1 1 5E8295EC
-P 4750 2650
-F 0 "U?" H 4600 2700 60  0000 L CNN
-F 1 "M1&M1W" H 4300 2850 60  0000 L CNN
-F 2 "" H 4750 2650 60  0000 C CNN
-F 3 "" H 4750 2650 60  0000 C CNN
-	1    4750 2650
-	1    0    0    -1
-$EndComp
-Text Label 5750 5600 1    50   ~ 0
+Text Label 2500 4100 1    50   ~ 0
 SPIO_CS1
 Wire Wire Line
-	5750 5150 5750 5600
-Wire Wire Line
-	5850 5150 5850 5600
-Wire Wire Line
-	5950 5150 5950 5600
-Wire Wire Line
-	6050 5150 6050 5600
-Wire Wire Line
-	6150 5150 6150 5600
-Text Label 5850 5600 1    50   ~ 0
+	2500 3650 2500 4100
+Wire Wire Line
+	2600 3650 2600 4100
+Wire Wire Line
+	2700 3650 2700 4100
+Wire Wire Line
+	2800 3650 2800 4100
+Wire Wire Line
+	2900 3650 2900 4100
+Text Label 2600 4100 1    50   ~ 0
 SPI0_MISO
-Text Label 5950 5600 1    50   ~ 0
+Text Label 2700 4100 1    50   ~ 0
 SPI0_SCLK
-Text Label 6050 5600 1    50   ~ 0
+Text Label 2800 4100 1    50   ~ 0
 SPI0_MOSI
-Text Label 6150 5600 1    50   ~ 0
+Text Label 2900 4100 1    50   ~ 0
 SPI0_CS0
 Entry Wire Line
@@
 Text HLabel 1100 6700 0    50   BiDi ~ 0
 COMM[3,0]
-Text Label 4300 2950 0    50   ~ 0
+Text Label 1050 1450 0    50   ~ 0
 TCK
-Text Label 4300 3050 0    50   ~ 0
+Text Label 1050 1550 0    50   ~ 0
 TDI
-Text Label 4300 3150 0    50   ~ 0
+Text Label 1050 1650 0    50   ~ 0
 TMS
-Text Label 4300 3250 0    50   ~ 0
+Text Label 1050 1750 0    50   ~ 0
 TDO
 Wire Wire Line
-	4300 2950 4550 2950
-Wire Wire Line
-	4300 3050 4550 3050
-Wire Wire Line
-	4300 3150 4550 3150
-Wire Wire Line
-	4300 3250 4550 3250
+	1050 1450 1300 1450
+Wire Wire Line
+	1050 1550 1300 1550
+Wire Wire Line
+	1050 1650 1300 1650
+Wire Wire Line
+	1050 1750 1300 1750
 Wire Bus Line
 	2650 6700 2400 6700
@@
 NRST
 Wire Wire Line
-	4550 3850 4300 3850
-Wire Wire Line
-	4550 3950 4300 3950
-Text HLabel 4300 3850 0    50   Input ~ 0
+	1300 2350 1050 2350
+Wire Wire Line
+	1300 2450 1050 2450
+Text HLabel 1050 2350 0    50   Input ~ 0
 RX_M1
-Text HLabel 4300 3950 0    50   Output ~ 0
+Text HLabel 1050 2450 0    50   Output ~ 0
 TX_M1
 $Comp
 L power:GND #PWR?
 U 1 1 5EB07062
-P 6950 5350
-F 0 "#PWR?" H 6950 5100 50  0001 C CNN
-F 1 "GND" H 6955 5177 50  0000 C CNN
-F 2 "" H 6950 5350 50  0001 C CNN
-F 3 "" H 6950 5350 50  0001 C CNN
-	1    6950 5350
+P 3700 3850
+F 0 "#PWR?" H 3700 3600 50  0001 C CNN
+F 1 "GND" H 3705 3677 50  0000 C CNN
+F 2 "" H 3700 3850 50  0001 C CNN
+F 3 "" H 3700 3850 50  0001 C CNN
+	1    3700 3850
 	1    0    0    -1
 $EndComp
@@
 L power:GND #PWR?
 U 1 1 5EB07767
-P 4850 5350
-F 0 "#PWR?" H 4850 5100 50  0001 C CNN
-F 1 "GND" H 4855 5177 50  0000 C CNN
-F 2 "" H 4850 5350 50  0001 C CNN
-F 3 "" H 4850 5350 50  0001 C CNN
-	1    4850 5350
+P 1600 3850
+F 0 "#PWR?" H 1600 3600 50  0001 C CNN
+F 1 "GND" H 1605 3677 50  0000 C CNN
+F 2 "" H 1600 3850 50  0001 C CNN
+F 3 "" H 1600 3850 50  0001 C CNN
+	1    1600 3850
 	1    0    0    -1
 $EndComp
@@
 L power:GND #PWR?
 U 1 1 5EB07C18
-P 6950 2300
-F 0 "#PWR?" H 6950 2050 50  0001 C CNN
-F 1 "GND" H 6955 2127 50  0000 C CNN
-F 2 "" H 6950 2300 50  0001 C CNN
-F 3 "" H 6950 2300 50  0001 C CNN
-	1    6950 2300
+P 3700 800
+F 0 "#PWR?" H 3700 550 50  0001 C CNN
+F 1 "GND" H 3705 627 50  0000 C CNN
+F 2 "" H 3700 800 50  0001 C CNN
+F 3 "" H 3700 800 50  0001 C CNN
+	1    3700 800
 	-1   0    0    1
 $EndComp
@@
 L power:GND #PWR?
 U 1 1 5EB09351
-P 7600 3450
-F 0 "#PWR?" H 7600 3200 50  0001 C CNN
-F 1 "GND" V 7605 3322 50  0000 R CNN
-F 2 "" H 7600 3450 50  0001 C CNN
-F 3 "" H 7600 3450 50  0001 C CNN
-	1    7600 3450
+P 4350 1950
+F 0 "#PWR?" H 4350 1700 50  0001 C CNN
+F 1 "GND" V 4355 1822 50  0000 R CNN
+F 2 "" H 4350 1950 50  0001 C CNN
+F 3 "" H 4350 1950 50  0001 C CNN
+	1    4350 1950
 	0    -1   -1   0
 $EndComp
 Wire Wire Line
-	7250 3450 7350 3450
-Wire Wire Line
-	7250 3350 7350 3350
-Wire Wire Line
-	7350 3350 7350 3450
-Connection ~ 7350 3450
-Wire Wire Line
-	7350 3450 7600 3450
-Wire Wire Line
-	6950 5350 6950 5150
-Wire Wire Line
-	4850 5150 4850 5350
-Wire Wire Line
-	6950 2450 6950 2300
+	4000 1950 4100 1950
+Wire Wire Line
+	4000 1850 4100 1850
+Wire Wire Line
+	4100 1850 4100 1950
+Connection ~ 4100 1950
+Wire Wire Line
+	4100 1950 4350 1950
+Wire Wire Line
+	3700 3850 3700 3650
+Wire Wire Line
+	1600 3650 1600 3850
+Wire Wire Line
+	3700 950  3700 800
 $Comp
 L Device:C C?
@@
 +5V_MCU
 Wire Wire Line
-	7250 3150 7550 3150
-Wire Wire Line
-	7550 3150 7550 3250
-Wire Wire Line
-	7550 3250 7250 3250
-Text Label 7500 3150 2    50   ~ 0
+	4000 1650 4300 1650
+Wire Wire Line
+	4300 1650 4300 1750
+Wire Wire Line
+	4300 1750 4000 1750
+Text Label 4250 1650 2    50   ~ 0
 +5V
-Text Label 7550 3050 2    50   ~ 0
+Text Label 4300 1550 2    50   ~ 0
 +1V8
-Text Label 7550 2950 2    50   ~ 0
+Text Label 4300 1450 2    50   ~ 0
 +3V3
 Wire Wire Line
-	7250 2950 7550 2950
-Wire Wire Line
-	7250 3050 7550 3050
+	4000 1450 4300 1450
+Wire Wire Line
+	4000 1550 4300 1550
 Connection ~ 10150 1200
 Wire Wire Line
@@
 L power:GND #PWR?
 U 1 1 5EB59EFD
-P 5050 2300
-F 0 "#PWR?" H 5050 2050 50  0001 C CNN
-F 1 "GND" H 5055 2127 50  0000 C CNN
-F 2 "" H 5050 2300 50  0001 C CNN
-F 3 "" H 5050 2300 50  0001 C CNN
-	1    5050 2300
-	-1   0    0    1
-$EndComp
-Wire Wire Line
-	5050 2450 5050 2300
+P 1800 800
+F 0 "#PWR?" H 1800 550 50  0001 C CNN
+F 1 "GND" H 1805 627 50  0000 C CNN
+F 2 "" H 1800 800 50  0001 C CNN
+F 3 "" H 1800 800 50  0001 C CNN
+	1    1800 800
+	-1   0    0    1
+$EndComp
+Wire Wire Line
+	1800 950  1800 800
+$Comp
+L M1&M1w:M1&M1W U?
+U 1 1 5E97DB3F
+P 1500 1150
+F 0 "U?" H 4044 53  60  0000 L CNN
+F 1 "M1&M1W" H 4044 -53 60  0000 L CNN
+F 2 "" H 1500 1150 60  0000 C CNN
+F 3 "" H 1500 1150 60  0000 C CNN
+	1    1500 1150
+	1    0    0    -1
+$EndComp
 Wire Bus Line
 	1300 6700 1300 7350

Commit message: Add files via upload
Parts:
- added C? (x4): 0.1u, symbol Device:C
- added D?: LED_RGB, symbol Device:LED_RGB
- added J?: Micro_SD_Card, symbol Connector:Micro_SD_Card
- added J? (x2): Conn_02x09_Odd_Even, symbol Connector_Generic:Conn_02x09_Odd_Even
- added R? (x2): 10k, symbol Device:R
- added R?: 10K, symbol Device:R
- added R? (x2): 2k, symbol Device:R
- added R?: 330, symbol Device:R
- added R? (x25): 33E, symbol Device:R
- added U?: DVP_PORT, symbol M1&M1w:DVP_PORT
- added U?: SMS, symbol pulse:SMS
Connections:
- net labels added: +1V5, +1V5_MCU, +2V8, +2V8_MCU, DVP_D0, DVP_D1, DVP_D2, DVP_D3, DVP_D4, DVP_D5, DVP_D6, DVP_D7, DVP_HSYNC, DVP_PCLK, DVP_PWDN, DVP_RST, DVP_SCL, DVP_SDA, DVP_VSYNC, DVP_XCLK, IO1, IO10, IO11, IO12, IO13, IO14, IO15, IO16, IO17, IO18, IO19, IO2, IO20, IO21, IO22, IO23, IO24, IO25, IO3, IO4, IO5, IO6, IO7, IO8, IO9, RGB_B, RGB_G, RGB_R, RST, SPI0_CS1
- wire segments 52 -> 250
- no-connect marks 0 -> 3
Other:
- moved on the sheet: C?

Commit message: Add files via upload
Parts:
- removed J? (x2): Conn_02x09_Odd_Even, symbol Connector_Generic:Conn_02x09_Odd_Even
- added C25: 0.1u, symbol Device:C
- added J5, J6: Conn_02x11_Odd_Even, Connector_PinHeader_2.54mm:PinHeader_2x11_P2.54mm_Vertical, symbol Connector_Generic:Conn_02x11_Odd_Even
- added R54: 10k, symbol Device:R
- added R77, R78, R79, R80, R84, R85, R86, R87: 33E, symbol Device:R
- added R88: 10K, symbol Device:R
- added U10: SMS, symbol pulse:SMS
- J7: renamed from J?; footprint (none) -> Connector_Card:microSD_HC_Wuerth_693072010801
- gave numbers to parts that had none: 43
Connections:
- net labels added: BOOT, I029, IO26, IO27, IO28, IO29, IO30, IO31, IO32, IO33
- net labels removed: TRST
- wire segments 250 -> 288
Other:
- note added: "Active Low"
- note added: "Switch abierto o cerrado"
- moved on the sheet: R62, R63, R71, R72, R73, R74, R75, R76, R81, R82, R83, R93
