File: AICE/sipeedm1w.sch (KiCad schematic (older format))
At the start: 58 parts, among them J5 Conn_02x11_Odd_Even, J6 Conn_02x11_Odd_Even, J7 Micro_SD_Card, U10 SMS, U11 DVP_PORT, U12 SMS, U9 M1&M1W

Commit message: Add files via upload
Parts:
- added R104, R105: 2K2, Resistor_SMD:R_0805_2012Metric_Pad1.15x1.40mm_HandSolder, symbol Device:R
- C25, C26, C27, C28, C29, C30, C31, C32, C33: footprint (none) -> Capacitor_SMD:C_0805_2012Metric_Pad1.15x1.40mm_HandSolder
- D6: footprint (none) -> LED_SMD:LED_RGB_Cree-PLCC-6_6x5mm_P2.1mm
- R54, R88, R90, R93, R94: footprint (none) -> Resistor_SMD:R_0603_1608Metric_Pad1.05x0.95mm_HandSolder
- R89: value 330 -> 2K2; footprint (none) -> Resistor_SMD:R_0805_2012Metric_Pad1.15x1.40mm_HandSolder
- R91, R92: value 2k -> 2k2; footprint (none) -> Resistor_SMD:R_0805_2012Metric_Pad1.15x1.40mm_HandSolder
- U11: footprint (none) -> Connector_FFC-FPC:Molex_200528-0240_1x24-1MP_P1.00mm_Horizontal
Connections:
- net GND: now also R104.2, R105.2
- net at D6.1 (RK), R89.1: no longer D6.2 (GK), D6.3 (BK)
- new net: D6.2 (GK), R104.1
- new net: D6.3 (BK), R105.1
Other:
- moved on the sheet: R89
Changed lines of the file:
@@
 F 0 "C29" V 8850 1300 50  0000 L CNN
 F 1 "0.1u" V 8850 1550 50  0000 L CNN
-F 2 "" H 8938 1350 50  0001 C CNN
+F 2 "Capacitor_SMD:C_0805_2012Metric_Pad1.15x1.40mm_HandSolder" H 8938 1350 50  0001 C CNN
 F 3 "~" H 8900 1500 50  0001 C CNN
 	1    8900 1500
@@
 F 0 "C30" V 9100 1300 50  0000 L CNN
 F 1 "0.1u" V 9100 1550 50  0000 L CNN
-F 2 "" H 9188 1350 50  0001 C CNN
+F 2 "Capacitor_SMD:C_0805_2012Metric_Pad1.15x1.40mm_HandSolder" H 9188 1350 50  0001 C CNN
 F 3 "~" H 9150 1500 50  0001 C CNN
 	1    9150 1500
@@
 F 0 "C31" V 9450 2300 50  0000 L CNN
 F 1 "0.1u" V 9450 2550 50  0000 L CNN
-F 2 "" H 9538 2350 50  0001 C CNN
+F 2 "Capacitor_SMD:C_0805_2012Metric_Pad1.15x1.40mm_HandSolder" H 9538 2350 50  0001 C CNN
 F 3 "~" H 9500 2500 50  0001 C CNN
 	1    9500 2500
@@
 F 0 "C32" V 9450 3100 50  0000 L CNN
 F 1 "0.1u" V 9450 3350 50  0000 L CNN
-F 2 "" H 9538 3150 50  0001 C CNN
+F 2 "Capacitor_SMD:C_0805_2012Metric_Pad1.15x1.40mm_HandSolder" H 9538 3150 50  0001 C CNN
 F 3 "~" H 9500 3300 50  0001 C CNN
 	1    9500 3300
@@
 F 0 "U9" H 1300 1400 60  0000 L CNN
 F 1 "M1&M1W" H 1150 1250 60  0000 L CNN
-F 2 "" H 1500 1150 60  0000 C CNN
+F 2 "" H 1500 1150 60  0001 C CNN
 F 3 "" H 1500 1150 60  0000 C CNN
 	1    1500 1150
@@
 F 0 "U11" H 5758 3975 50  0000 C CNN
 F 1 "DVP_PORT" H 5758 3884 50  0000 C CNN
-F 2 "" H 5700 3900 50  0001 C CNN
+F 2 "Connector_FFC-FPC:Molex_200528-0240_1x24-1MP_P1.00mm_Horizontal" H 5700 3900 50  0001 C CNN
 F 3 "" H 5700 3900 50  0001 C CNN
 	1    5750 2550
@@
 F 0 "C33" V 9650 2300 50  0000 L CNN
 F 1 "0.1u" V 9650 2550 50  0000 L CNN
-F 2 "" H 9738 2350 50  0001 C CNN
+F 2 "Capacitor_SMD:C_0805_2012Metric_Pad1.15x1.40mm_HandSolder" H 9738 2350 50  0001 C CNN
 F 3 "~" H 9700 2500 50  0001 C CNN
 	1    9700 2500
@@
 F 0 "R90" V 6400 5200 50  0000 L CNN
 F 1 "10K" V 6350 5050 50  0000 L CNN
-F 2 "" V 6280 5100 50  0001 C CNN
+F 2 "Resistor_SMD:R_0603_1608Metric_Pad1.05x0.95mm_HandSolder" V 6280 5100 50  0001 C CNN
 F 3 "~" H 6350 5100 50  0001 C CNN
 	1    6350 5100
@@
 F 0 "C26" H 7615 5596 50  0000 L CNN
 F 1 "0.1u" H 7615 5505 50  0000 L CNN
-F 2 "" H 7538 5400 50  0001 C CNN
+F 2 "Capacitor_SMD:C_0805_2012Metric_Pad1.15x1.40mm_HandSolder" H 7538 5400 50  0001 C CNN
 F 3 "~" H 7500 5550 50  0001 C CNN
 	1    7500 5550
@@
 F 0 "C28" V 8150 3100 50  0000 L CNN
 F 1 "0.1u" V 8150 3350 50  0000 L CNN
-F 2 "" H 8238 3150 50  0001 C CNN
+F 2 "Capacitor_SMD:C_0805_2012Metric_Pad1.15x1.40mm_HandSolder" H 8238 3150 50  0001 C CNN
 F 3 "~" H 8200 3300 50  0001 C CNN
 	1    8200 3300
@@
 F 0 "C27" V 8150 2300 50  0000 L CNN
 F 1 "0.1u" V 8150 2550 50  0000 L CNN
-F 2 "" H 8238 2350 50  0001 C CNN
+F 2 "Capacitor_SMD:C_0805_2012Metric_Pad1.15x1.40mm_HandSolder" H 8238 2350 50  0001 C CNN
 F 3 "~" H 8200 2500 50  0001 C CNN
 	1    8200 2500
@@
 P 6650 3450
 F 0 "R92" V 6700 3250 50  0000 C CNN
-F 1 "2k" V 6650 3450 50  0000 C CNN
-F 2 "" V 6580 3450 50  0001 C CNN
+F 1 "2k2" V 6650 3450 50  0000 C CNN
+F 2 "Resistor_SMD:R_0805_2012Metric_Pad1.15x1.40mm_HandSolder" V 6580 3450 50  0001 C CNN
 F 3 "~" H 6650 3450 50  0001 C CNN
 	1    6650 3450
@@
 P 6650 3250
 F 0 "R91" V 6700 3050 50  0000 C CNN
-F 1 "2k" V 6650 3250 50  0000 C CNN
-F 2 "" V 6580 3250 50  0001 C CNN
+F 1 "2k2" V 6650 3250 50  0000 C CNN
+F 2 "Resistor_SMD:R_0805_2012Metric_Pad1.15x1.40mm_HandSolder" V 6580 3250 50  0001 C CNN
 F 3 "~" H 6650 3250 50  0001 C CNN
 	1    6650 3250
@@
 F 0 "D6" V 5496 4870 50  0000 R CNN
 F 1 "LED_RGB" V 5405 4870 50  0000 R CNN
-F 2 "" H 5450 5150 50  0001 C CNN
+F 2 "LED_SMD:LED_RGB_Cree-PLCC-6_6x5mm_P2.1mm" H 5450 5150 50  0001 C CNN
 F 3 "~" H 5450 5150 50  0001 C CNN
 	1    5450 5200
@@
 Wire Wire Line
 	5250 5400 5250 5550
-Wire Wire Line
-	5250 5550 5450 5550
-Wire Wire Line
-	5650 5550 5650 5400
-Wire Wire Line
-	5450 5400 5450 5550
-Connection ~ 5450 5550
-Wire Wire Line
-	5450 5550 5650 5550
 $Comp
 L Device:R R?
 U 1 1 5ECA3509
-P 5450 5800
+P 5250 5700
 AR Path="/5E829221/5ECA3509" Ref="R?"  Part="1"
 AR Path="/5E828FD1/5ECA3509" Ref="R89"  Part="1"
-F 0 "R89" H 5520 5846 50  0000 L CNN
-F 1 "330" H 5520 5755 50  0000 L CNN
-F 2 "" V 5380 5800 50  0001 C CNN
-F 3 "~" H 5450 5800 50  0001 C CNN
-	1    5450 5800
+F 0 "R89" V 5200 5800 50  0000 L CNN
+F 1 "2K2" V 5250 5600 50  0000 L CNN
+F 2 "Resistor_SMD:R_0805_2012Metric_Pad1.15x1.40mm_HandSolder" V 5180 5700 50  0001 C CNN
+F 3 "~" H 5250 5700 50  0001 C CNN
+	1    5250 5700
 	1    0    0    -1
 $EndComp
@@
 L power:GND #PWR?
 U 1 1 5ECA350F
-P 5450 6050
+P 5250 5950
 AR Path="/5E829221/5ECA350F" Ref="#PWR?"  Part="1"
 AR Path="/5E828FD1/5ECA350F" Ref="#PWR041"  Part="1"
-F 0 "#PWR041" H 5450 5800 50  0001 C CNN
-F 1 "GND" H 5455 5877 50  0000 C CNN
-F 2 "" H 5450 6050 50  0001 C CNN
-F 3 "" H 5450 6050 50  0001 C CNN
-	1    5450 6050
-	1    0    0    -1
-$EndComp
-Wire Wire Line
-	5450 5650 5450 5550
-Wire Wire Line
-	5450 6050 5450 5950
+F 0 "#PWR041" H 5250 5700 50  0001 C CNN
+F 1 "GND" H 5255 5777 50  0000 C CNN
+F 2 "" H 5250 5950 50  0001 C CNN
+F 3 "" H 5250 5950 50  0001 C CNN
+	1    5250 5950
+	1    0    0    -1
+$EndComp
+Wire Wire Line
+	5250 5950 5250 5850
 Text Label 5250 4700 3    50   ~ 0
 RGB_R
@@
 F 0 "R94" V 8650 5550 50  0000 C CNN
 F 1 "10k" V 8600 5750 50  0000 C CNN
-F 2 "" V 8530 5750 50  0001 C CNN
+F 2 "Resistor_SMD:R_0603_1608Metric_Pad1.05x0.95mm_HandSolder" V 8530 5750 50  0001 C CNN
 F 3 "~" H 8600 5750 50  0001 C CNN
 	1    8600 5750
@@
 F 0 "R54" V 800 3050 50  0000 C CNN
 F 1 "10k" V 750 3250 50  0000 C CNN
-F 2 "" V 680 3250 50  0001 C CNN
+F 2 "Resistor_SMD:R_0603_1608Metric_Pad1.05x0.95mm_HandSolder" V 680 3250 50  0001 C CNN
 F 3 "~" H 750 3250 50  0001 C CNN
 	1    750  3250
@@
 F 0 "C25" H 6265 6946 50  0000 L CNN
 F 1 "0.1u" H 6265 6855 50  0000 L CNN
-F 2 "" H 6188 6750 50  0001 C CNN
+F 2 "Capacitor_SMD:C_0805_2012Metric_Pad1.15x1.40mm_HandSolder" H 6188 6750 50  0001 C CNN
 F 3 "~" H 6150 6900 50  0001 C CNN
 	1    6150 6900
@@
 F 0 "R88" V 5100 6750 50  0000 L CNN
 F 1 "10K" V 5050 6600 50  0000 L CNN
-F 2 "" V 4980 6650 50  0001 C CNN
+F 2 "Resistor_SMD:R_0603_1608Metric_Pad1.05x0.95mm_HandSolder" V 4980 6650 50  0001 C CNN
 F 3 "~" H 5050 6650 50  0001 C CNN
 	1    5050 6650
@@
 F 0 "R93" V 8700 5150 50  0000 C CNN
 F 1 "10k" V 8650 5350 50  0000 C CNN
-F 2 "" V 8580 5350 50  0001 C CNN
+F 2 "Resistor_SMD:R_0603_1608Metric_Pad1.05x0.95mm_HandSolder" V 8580 5350 50  0001 C CNN
 F 3 "~" H 8650 5350 50  0001 C CNN
 	1    8650 5350
@@
 	1    0    0    -1
 $EndComp
+Wire Wire Line
+	5450 5400 5450 5550
+$Comp
+L Device:R R?
+U 1 1 5EB2A360
+P 5450 5700
+AR Path="/5E829221/5EB2A360" Ref="R?"  Part="1"
+AR Path="/5E828FD1/5EB2A360" Ref="R104"  Part="1"
+F 0 "R104" V 5400 5800 50  0000 L CNN
+F 1 "2K2" V 5450 5600 50  0000 L CNN
+F 2 "Resistor_SMD:R_0805_2012Metric_Pad1.15x1.40mm_HandSolder" V 5380 5700 50  0001 C CNN
+F 3 "~" H 5450 5700 50  0001 C CNN
+	1    5450 5700
+	1    0    0    -1
+$EndComp
+$Comp
+L power:GND #PWR?
+U 1 1 5EB2A366
+P 5450 5950
+AR Path="/5E829221/5EB2A366" Ref="#PWR?"  Part="1"
+AR Path="/5E828FD1/5EB2A366" Ref="#PWR0104"  Part="1"
+F 0 "#PWR0104" H 5450 5700 50  0001 C CNN
+F 1 "GND" H 5455 5777 50  0000 C CNN
+F 2 "" H 5450 5950 50  0001 C CNN
+F 3 "" H 5450 5950 50  0001 C CNN
+	1    5450 5950
+	1    0    0    -1
+$EndComp
+Wire Wire Line
+	5450 5950 5450 5850
+Wire Wire Line
+	5650 5400 5650 5550
+$Comp
+L Device:R R?
+U 1 1 5EB44F51
+P 5650 5700
+AR Path="/5E829221/5EB44F51" Ref="R?"  Part="1"
+AR Path="/5E828FD1/5EB44F51" Ref="R105"  Part="1"
+F 0 "R105" V 5600 5800 50  0000 L CNN
+F 1 "2K2" V 5650 5600 50  0000 L CNN
+F 2 "Resistor_SMD:R_0805_2012Metric_Pad1.15x1.40mm_HandSolder" V 5580 5700 50  0001 C CNN
+F 3 "~" H 5650 5700 50  0001 C CNN
+	1    5650 5700
+	1    0    0    -1
+$EndComp
+$Comp
+L power:GND #PWR?
+U 1 1 5EB44F57
+P 5650 5950
+AR Path="/5E829221/5EB44F57" Ref="#PWR?"  Part="1"
+AR Path="/5E828FD1/5EB44F57" Ref="#PWR0105"  Part="1"
+F 0 "#PWR0105" H 5650 5700 50  0001 C CNN
+F 1 "GND" H 5655 5777 50  0000 C CNN
+F 2 "" H 5650 5950 50  0001 C CNN
+F 3 "" H 5650 5950 50  0001 C CNN
+	1    5650 5950
+	1    0    0    -1
+$EndComp
+Wire Wire Line
+	5650 5950 5650 5850
 Wire Bus Line
 	1650 6700 1650 7350

Commit message: Add files via upload
Parts:
- U10: footprint (none) -> Connector_PinHeader_2.54mm:PinHeader_2x02_P2.54mm_Vertical
- U11: footprint Connector_FFC-FPC:Molex_200528-0240_1x24-1MP_P1.00mm_Horizontal -> Connector_FFC-FPC:Molex_502244-2430_1x24-1MP_P0.5mm_Horizontal
- U12: footprint (none) -> AICE:SMS_BUTTON
- U9: footprint (none) -> AICE:QFN-72_25.4x25.4_Pitch1.27mm
Changed lines of the file:
@@
 F 0 "U9" H 1300 1400 60  0000 L CNN
 F 1 "M1&M1W" H 1150 1250 60  0000 L CNN
-F 2 "" H 1500 1150 60  0001 C CNN
+F 2 "AICE:QFN-72_25.4x25.4_Pitch1.27mm" H 1500 1150 60  0001 C CNN
 F 3 "" H 1500 1150 60  0000 C CNN
 	1    1500 1150
@@
 F 0 "U11" H 5758 3975 50  0000 C CNN
 F 1 "DVP_PORT" H 5758 3884 50  0000 C CNN
-F 2 "Connector_FFC-FPC:Molex_200528-0240_1x24-1MP_P1.00mm_Horizontal" H 5700 3900 50  0001 C CNN
+F 2 "Connector_FFC-FPC:Molex_502244-2430_1x24-1MP_P0.5mm_Horizontal" H 5700 3900 50  0001 C CNN
 F 3 "" H 5700 3900 50  0001 C CNN
 	1    5750 2550
@@
 F 0 "U12" H 6900 5975 50  0000 C CNN
 F 1 "SMS" H 6900 5884 50  0000 C CNN
-F 2 "" H 7300 5900 50  0001 C CNN
+F 2 "AICE:SMS_BUTTON" H 7300 5900 50  0001 C CNN
 F 3 "" H 7300 5900 50  0001 C CNN
 	1    6900 5700
@@
 F 0 "U10" H 5550 7325 50  0000 C CNN
 F 1 "SMS" H 5550 7234 50  0000 C CNN
-F 2 "" H 5950 7250 50  0001 C CNN
+F 2 "Connector_PinHeader_2.54mm:PinHeader_2x02_P2.54mm_Vertical" H 5950 7250 50  0001 C CNN
 F 3 "" H 5950 7250 50  0001 C CNN
 	1    5550 7050

Commit message: Add files via upload
Parts:
- removed R55, R56, R57, R58, R59, R60, R61, R62, R63, R64, R65, R66, R67, R68, R69, R70, R71, R72, R73, R74, R75, R76, R77, R78, R79, R80, R81, R82, R83, R84, R85, R86, R87: 33E, symbol Device:R
- C25, C27, C28, C29, C30, C31, C32, C33: footprint Capacitor_SMD:C_0805_2012Metric_Pad1.15x1.40mm_HandSolder -> Capacitor_SMD:C_0603_1608Metric_Pad1.05x0.95mm_HandSolder
- C26: footprint Capacitor_SMD:C_0805_2012Metric_Pad1.15x1.40mm_HandSolder -> Capacitor_SMD:C_0603_1608Metric
- R104, R105, R89, R91, R92: footprint Resistor_SMD:R_0805_2012Metric_Pad1.15x1.40mm_HandSolder -> Resistor_SMD:R_0603_1608Metric_Pad1.05x0.95mm_HandSolder
Connections:
- net SPIO_CS1 is gone; now on net SPI0_CS1: U9.26 (IO25)
- net IO1: now also J5.5 (Pin_5)
- net IO10: now also J5.14 (Pin_14)
- net IO11: now also J5.15 (Pin_15)
- net IO12: now also J5.16 (Pin_16)
- net IO13: now also J5.17 (Pin_17)
- net IO14: now also J5.18 (Pin_18)
- net IO15: now also J5.19 (Pin_19)
- net IO16: now also J5.20 (Pin_20)
- net IO17: now also J5.21 (Pin_21)
- net IO18: now also J5.22 (Pin_22)
- net IO19: now also J6.5 (Pin_5)
- net IO2: now also J5.6 (Pin_6)
- net IO20: now also J6.6 (Pin_6)
- net IO21: now also J6.7 (Pin_7)
- net IO22: now also J6.8 (Pin_8)
- net IO23: now also J6.9 (Pin_9)
- net IO24: now also J6.10 (Pin_10)
- net IO25: now also J6.11 (Pin_11)
- net IO26: now also J6.12 (Pin_12)
- net IO27: now also J6.13 (Pin_13)
- net IO28: now also J6.14 (Pin_14)
- net IO29: now also J6.15 (Pin_15)
- net IO3: now also J5.7 (Pin_7)
- net IO30: now also J6.16 (Pin_16)
- net IO31: now also J6.17 (Pin_17)
- net IO32: now also J6.18 (Pin_18)
- net IO33: now also J6.19 (Pin_19)
- net IO4: now also J5.8 (Pin_8)
- net IO5: now also J5.9 (Pin_9)
- net IO6: now also J5.10 (Pin_10)
- net IO7: now also J5.11 (Pin_11)
- net IO8: now also J5.12 (Pin_12)
- net IO9: now also J5.13 (Pin_13)
