File: AICE/sipeedm1w.sch (KiCad schematic (older format))
At the start: 27 parts, among them J5 Conn_02x11_Odd_Even, J6 Conn_02x11_Odd_Even, J7 Micro_SD_Card, U10 SMS, U11 DVP_PORT, U12 SMS, U9 M1&M1W

Commit message: Add files via upload
Parts:
- added C61: 0.1u, Capacitor_SMD:C_0603_1608Metric_Pad1.05x0.95mm_HandSolder, symbol Device:C
Connections:
- net +1V8_MCU: now also C61.2
- net GND: now also C61.1
Changed lines of the file:
@@
 $EndComp
 Wire Wire Line
-	9500 3050 9850 3050
+	9500 3050 9750 3050
 Connection ~ 9500 3050
 $Comp
@@
 Entry Wire Line
 	3000 7350 3100 7450
+$Comp
+L Device:C C?
+U 1 1 5EB890D2
+P 9750 3300
+AR Path="/5E829221/5EB890D2" Ref="C?"  Part="1"
+AR Path="/5E828FD1/5EB890D2" Ref="C61"  Part="1"
+F 0 "C61" V 9700 3100 50  0000 L CNN
+F 1 "0.1u" V 9700 3350 50  0000 L CNN
+F 2 "Capacitor_SMD:C_0603_1608Metric_Pad1.05x0.95mm_HandSolder" H 9788 3150 50  0001 C CNN
+F 3 "~" H 9750 3300 50  0001 C CNN
+	1    9750 3300
+	-1   0    0    1
+$EndComp
+Wire Wire Line
+	9750 3150 9750 3050
+Wire Wire Line
+	9750 3450 9750 3600
+$Comp
+L power:GND #PWR078
+U 1 1 5EB890DA
+P 9750 3600
+F 0 "#PWR078" H 9750 3350 50  0001 C CNN
+F 1 "GND" H 9755 3427 50  0000 C CNN
+F 2 "" H 9750 3600 50  0001 C CNN
+F 3 "" H 9750 3600 50  0001 C CNN
+	1    9750 3600
+	1    0    0    -1
+$EndComp
 Wire Bus Line
 	3000 6700 3000 7350
 Wire Bus Line
 	1650 6700 1650 7350
+Connection ~ 9750 3050
+Wire Wire Line
+	9750 3050 9850 3050
 $EndSCHEMATC

Commit message: Add files via upload
Parts:
- removed J5, J6: Conn_02x11_Odd_Even, Connector_PinHeader_2.54mm:PinHeader_2x11_P2.54mm_Vertical, symbol Connector_Generic:Conn_02x11_Odd_Even
- added J5, J6: Conn_02x10_Odd_Even, Connector_PinHeader_2.54mm:PinHeader_2x10_P2.54mm_Vertical, symbol Connector_Generic:Conn_02x10_Odd_Even
- C25, C27, C28, C29, C30, C31, C32, C33, C61: footprint Capacitor_SMD:C_0603_1608Metric_Pad1.05x0.95mm_HandSolder -> Capacitor_SMD:C_0603_1608Metric
- R104, R105, R54, R88, R89, R90, R91, R92, R93, R94: footprint Resistor_SMD:R_0603_1608Metric_Pad1.05x0.95mm_HandSolder -> Resistor_SMD:R_0603_1608Metric
Connections:
- net +3V3_MCU: now also J5.1 (Pin_1), J5.3 (Pin_3), J6.19 (Pin_19)
- net COMM0: now also U9.59 (D4); no longer U9.27 (IO26)
- net COMM1: now also U9.60 (D3); no longer U9.28 (IO27)
- net COMM2: now also U9.61 (D2); no longer U9.29 (IO28)
- net COMM3: now also U9.62 (D1); no longer U9.30 (IO29)
- net DVP_D0: now also U9.36 (IO35); no longer U9.71 (D0)
- net DVP_D1: now also U9.34 (IO33); no longer U9.70 (D1)
- net DVP_D2: now also U9.33 (IO32); no longer U9.69 (D2)
- net DVP_D3: now also U9.35 (IO34); no longer U9.68 (D3)
- net DVP_D4: now also U9.37 (IO36); no longer U9.67 (D4)
- net DVP_D5: now also U9.39 (IO38); no longer U9.66 (D5)
- net DVP_D6: now also U9.40 (IO39); no longer U9.65 (D6)
- net DVP_D7: now also U9.42 (IO41); no longer U9.64 (D7)
- net DVP_HSYNC: now also U9.43 (IO42); no longer U9.46 (IO45)
- net DVP_PCLK: now also U9.38 (IO37); no longer U9.48 (IO47)
- net DVP_PWDN: now also U9.44 (IO43); no longer U9.45 (IO44)
- net DVP_RST: now also U9.46 (IO45); no longer U9.43 (IO42)
- net DVP_SCL: now also U9.47 (IO46); no longer U9.42 (IO41)
- net DVP_SDA: now also U9.48 (IO47); no longer U9.41 (IO40)
- net DVP_VSYNC: now also U9.45 (IO44); no longer U9.44 (IO43)
- net DVP_XCLK: now also U9.41 (IO40); no longer U9.47 (IO46)
- net GND: now also J5.2 (Pin_2), J5.4 (Pin_4), J6.18 (Pin_18), J6.20 (Pin_20)
- net IO1: now also U9.32 (IO31), J5.5 (Pin_5); no longer U9.19 (IO18)
- net IO10: now also U9.23 (IO22), J5.14 (Pin_14); no longer U9.33 (IO32)
- net IO11: now also U9.22 (IO21), J5.15 (Pin_15); no longer U9.34 (IO33)
- net IO12: now also U9.21 (IO20), J5.16 (Pin_16); no longer U9.35 (IO34)
- net IO13: now also U9.20 (IO19), J5.17 (Pin_17); no longer U9.36 (IO35)
- net IO14: now also U9.19 (IO18), J5.18 (Pin_18); no longer U9.37 (IO36)
- net IO15: now also U9.18 (IO17), J5.19 (Pin_19); no longer U9.38 (IO37)
- net IO16: now also U9.16 (IO15), J5.20 (Pin_20); no longer U9.39 (IO38)
- net IO17: now also U9.15 (IO14), J6.1 (Pin_1); no longer U9.40 (IO39)
- net IO18: now also U9.14 (IO13), J6.2 (Pin_2); no longer U9.56 (D7)
- net IO19: now also U9.13 (IO12), J6.3 (Pin_3); no longer U9.57 (D6)
- net IO2: now also U9.31 (IO30), J5.6 (Pin_6); no longer U9.20 (IO19)
- net IO20: now also U9.12 (IO11), J6.4 (Pin_4); no longer U9.58 (D5)
- net IO21: now also U9.11 (IO10), J6.5 (Pin_5); no longer U9.59 (D4)
- net IO22: now also U9.10 (IO9), J6.6 (Pin_6); no longer U9.60 (D3)
- net IO23: now also U9.9 (IO8), J6.7 (Pin_7); no longer U9.61 (D2)
- net IO24: now also U9.8 (IO7), J6.8 (Pin_8); no longer U9.62 (D1)
- net IO25: now also U9.7 (IO6), J6.9 (Pin_9); no longer U9.63 (D0)
- net IO26: now also U9.6 (IO5), J6.10 (Pin_10); no longer U9.5 (IO4)
- net IO27: now also U9.5 (IO4), J6.11 (Pin_11); no longer U9.6 (IO5)
- net IO28: now also U9.66 (D5), J6.12 (Pin_12); no longer U9.9 (IO8)
- net IO29: now also U9.67 (D4), J6.13 (Pin_13); no longer U9.10 (IO9)
- net IO3: now also U9.30 (IO29), J5.7 (Pin_7); no longer U9.21 (IO20)
- net IO30: now also U9.68 (D3), J6.14 (Pin_14); no longer U9.11 (IO10)
- net IO31: now also U9.69 (D2), J6.15 (Pin_15); no longer U9.12 (IO11)
- net IO32: now also U9.70 (D1), J6.16 (Pin_16); no longer U9.16 (IO15)
- net IO33: now also U9.71 (D0), J6.17 (Pin_17); no longer U9.18 (IO17)
- net IO4: now also U9.29 (IO28), J5.8 (Pin_8); no longer U9.22 (IO21)
- net IO5: now also U9.28 (IO27), J5.9 (Pin_9); no longer U9.23 (IO22)
- net IO6: now also U9.27 (IO26), J5.10 (Pin_10); no longer U9.24 (IO23)
- net IO7: now also U9.26 (IO25), J5.11 (Pin_11); no longer U9.25 (IO24)
- net IO8: now also U9.25 (IO24), J5.12 (Pin_12); no longer U9.31 (IO30)
- net IO9: now also U9.24 (IO23), J5.13 (Pin_13); no longer U9.32 (IO31)
- net RGB_B: now also U9.58 (D5); no longer U9.14 (IO13)
- net RGB_G: now also U9.57 (D6); no longer U9.13 (IO12)
- net RGB_R: now also U9.56 (D7); no longer U9.15 (IO14)
- net RX_M1: now also U9.64 (D7); no longer U9.7 (IO6)
- net SPI0_CS1: now also U9.63 (D0); no longer U9.26 (IO25)
- net TX_M1: now also U9.65 (D6); no longer U9.8 (IO7)
Other:
- moved on the sheet: R54, U9

Commit message: Add files via upload
Parts:
- removed C25: 0.1u, Capacitor_SMD:C_0603_1608Metric, symbol Device:C
- removed R88: 10K, Resistor_SMD:R_0603_1608Metric, symbol Device:R
- removed U10: SMS, Connector_PinHeader_2.54mm:PinHeader_2x02_P2.54mm_Vertical, symbol pulse:SMS
- U11: footprint Connector_FFC-FPC:Molex_502244-2430_1x24-1MP_P0.5mm_Horizontal -> Connector_FFC-FPC:Molex_502231-2400_1x24-1SH_P0.5mm_Vertical
Connections:
- net RGB_B: now also U9.56 (D7); no longer U9.58 (D5)
- net RGB_R: now also U9.58 (D5); no longer U9.56 (D7)
Changed lines of the file:
@@
 F 0 "U11" H 5758 3975 50  0000 C CNN
 F 1 "DVP_PORT" H 5758 3884 50  0000 C CNN
-F 2 "Connector_FFC-FPC:Molex_502244-2430_1x24-1MP_P0.5mm_Horizontal" H 5700 3900 50  0001 C CNN
+F 2 "Connector_FFC-FPC:Molex_502231-2400_1x24-1SH_P0.5mm_Vertical" H 5700 3900 50  0001 C CNN
 F 3 "" H 5700 3900 50  0001 C CNN
 	1    5750 2550
@@
 Wire Wire Line
 	5250 4700 5250 5000
-Text Label 3400 850  3    50   ~ 0
+Text Label 3200 850  3    50   ~ 0
 RGB_R
 Text Label 3300 850  3    50   ~ 0
 RGB_G
-Text Label 3200 850  3    50   ~ 0
+Text Label 3400 850  3    50   ~ 0
 RGB_B
 Wire Wire Line
+	3400 850  3400 1150
+Wire Wire Line
+	3300 850  3300 1150
+Wire Wire Line
 	3200 850  3200 1150
-Wire Wire Line
-	3300 850  3300 1150
-Wire Wire Line
-	3400 850  3400 1150
 Text Label 3500 800  3    50   ~ 0
 RST
@@
 Wire Wire Line
 	750  3250 1300 3250
-$Comp
-L pulse:SMS U?
-U 1 1 5EA9A7E7
-P 5550 7050
-AR Path="/5E829221/5EA9A7E7" Ref="U?"  Part="1"
-AR Path="/5E828FD1/5EA9A7E7" Ref="U10"  Part="1"
-F 0 "U10" H 5550 7325 50  0000 C CNN
-F 1 "SMS" H 5550 7234 50  0000 C CNN
-F 2 "Connector_PinHeader_2.54mm:PinHeader_2x02_P2.54mm_Vertical" H 5950 7250 50  0001 C CNN
-F 3 "" H 5950 7250 50  0001 C CNN
-	1    5550 7050
-	1    0    0    -1
-$EndComp
-Wire Wire Line
-	5300 7000 5300 6650
-Wire Wire Line
-	5300 6650 5800 6650
-Wire Wire Line
-	5800 7000 5800 6650
-Connection ~ 5800 6650
-Wire Wire Line
-	5800 6650 6150 6650
-$Comp
-L power:GND #PWR?
-U 1 1 5EA9A7F2
-P 5300 7300
-AR Path="/5E829221/5EA9A7F2" Ref="#PWR?"  Part="1"
-AR Path="/5E828FD1/5EA9A7F2" Ref="#PWR040"  Part="1"
-F 0 "#PWR040" H 5300 7050 50  0001 C CNN
-F 1 "GND" H 5305 7127 50  0000 C CNN
-F 2 "" H 5300 7300 50  0001 C CNN
-F 3 "" H 5300 7300 50  0001 C CNN
-	1    5300 7300
-	1    0    0    -1
-$EndComp
-$Comp
-L power:GND #PWR?
-U 1 1 5EA9A7F8
-P 5800 7300
-AR Path="/5E829221/5EA9A7F8" Ref="#PWR?"  Part="1"
-AR Path="/5E828FD1/5EA9A7F8" Ref="#PWR042"  Part="1"
-F 0 "#PWR042" H 5800 7050 50  0001 C CNN
-F 1 "GND" H 5805 7127 50  0000 C CNN
-F 2 "" H 5800 7300 50  0001 C CNN
-F 3 "" H 5800 7300 50  0001 C CNN
-	1    5800 7300
-	1    0    0    -1
-$EndComp
-Wire Wire Line
-	5800 7300 5800 7150
-Wire Wire Line
-	5300 7150 5300 7300
-$Comp
-L power:GND #PWR?
-U 1 1 5EA9A800
-P 6150 7150
-AR Path="/5E829221/5EA9A800" Ref="#PWR?"  Part="1"
-AR Path="/5E828FD1/5EA9A800" Ref="#PWR043"  Part="1"
-F 0 "#PWR043" H 6150 6900 50  0001 C CNN
-F 1 "GND" H 6155 6977 50  0000 C CNN
-F 2 "" H 6150 7150 50  0001 C CNN
-F 3 "" H 6150 7150 50  0001 C CNN
-	1    6150 7150
-	1    0    0    -1
-$EndComp
-Wire Wire Line
-	6150 6750 6150 6650
-Connection ~ 6150 6650
-Wire Wire Line
-	6150 7050 6150 7150
-$Comp
-L Device:C C?
-U 1 1 5EA9A809
-P 6150 6900
-AR Path="/5E829221/5EA9A809" Ref="C?"  Part="1"
-AR Path="/5E828FD1/5EA9A809" Ref="C25"  Part="1"
-F 0 "C25" H 6265 6946 50  0000 L CNN
-F 1 "0.1u" H 6265 6855 50  0000 L CNN
-F 2 "Capacitor_SMD:C_0603_1608Metric" H 6188 6750 50  0001 C CNN
-F 3 "~" H 6150 6900 50  0001 C CNN
-	1    6150 6900
-	1    0    0    -1
-$EndComp
-Wire Wire Line
-	6150 6650 6600 6650
-Text Label 4550 6650 0    50   ~ 0
-+3V3
-Text Label 6600 6650 2    50   ~ 0
-BOOT
-$Comp
-L Device:R R?
-U 1 1 5EA9A7DF
-P 5050 6650
-AR Path="/5E926AEA/5EA9A7DF" Ref="R?"  Part="1"
-AR Path="/5E829221/5EA9A7DF" Ref="R?"  Part="1"
-AR Path="/5E828FD1/5EA9A7DF" Ref="R88"  Part="1"
-F 0 "R88" V 5100 6750 50  0000 L CNN
-F 1 "10K" V 5050 6600 50  0000 L CNN
-F 2 "Resistor_SMD:R_0603_1608Metric" V 4980 6650 50  0001 C CNN
-F 3 "~" H 5050 6650 50  0001 C CNN
-	1    5050 6650
-	0    -1   -1   0
-$EndComp
-Wire Wire Line
-	5200 6650 5300 6650
-Connection ~ 5300 6650
-Wire Wire Line
-	4550 6650 4900 6650
 Wire Notes Line
 	550  6500 4350 6500
