File: AICE/omega.sch (KiCad schematic (older format))
At the start: 5 parts

Commit message: Add files via upload
Parts:
- added R?: R, symbol Device:R
Connections:
- net at U?.14 (1/I2S_SDO): now also R?.1
- new net FPGA_RST: R?.2
Changed lines of the file:
@@
 SPI_CS1
-Entry Wire Line
-	3600 7000 3700 7100
-Entry Wire Line
-	3600 6900 3700 7000
 Entry Wire Line
 	3600 6800 3700 6900
 Entry Wire Line
 	3600 6700 3700 6800
+Entry Wire Line
+	3600 6600 3700 6700
+Text Label 3750 6700 0    50   ~ 0
+OmSPI0
 Text Label 3750 6800 0    50   ~ 0
-OmSPI0
+OmSPI1
 Text Label 3750 6900 0    50   ~ 0
-OmSPI1
-Text Label 3750 7000 0    50   ~ 0
 OmSPI2
-Text Label 3750 7100 0    50   ~ 0
-OmSPI3
+Wire Wire Line
+	3700 6700 4600 6700
 Wire Wire Line
 	3700 6800 4600 6800
 Wire Wire Line
 	3700 6900 4600 6900
-Wire Wire Line
-	3700 7000 4600 7000
-Wire Wire Line
-	3700 7100 4600 7100
+Text Label 4600 6700 2    50   ~ 0
+SPI_MISO
 Text Label 4600 6800 2    50   ~ 0
-SPI_MISO
+SPI_CLK
 Text Label 4600 6900 2    50   ~ 0
-SPI_CLK
-Text Label 4600 7000 2    50   ~ 0
 SPI_MOSI
-Text Label 4600 7100 2    50   ~ 0
-SPI_CS1
 Wire Bus Line
-	3600 6250 3350 6250
-Text HLabel 3350 6250 0    50   BiDi ~ 0
-OmSPI[3,0]
+	3600 6150 3350 6150
+Text HLabel 3350 6150 0    50   BiDi ~ 0
+OmSPI[4,0]
 Text HLabel 6350 3550 2    50   Input ~ 0
 RX_OM
@@
 Wire Wire Line
 	4650 3550 4350 3550
+Wire Wire Line
+	3700 7100 4600 7100
+Entry Wire Line
+	3600 7000 3700 7100
+Text Label 4600 7000 2    50   ~ 0
+SPI_CS1
+Wire Wire Line
+	3700 7000 4600 7000
+Text Label 3750 7000 0    50   ~ 0
+OmSPI3
+Entry Wire Line
+	3600 6900 3700 7000
+Text Label 3750 7100 0    50   ~ 0
+OmSPI4
+Text Label 3550 3950 0    50   ~ 0
+FPGA_RST
+$Comp
+L Device:R R?
+U 1 1 5E87BB84
+P 4200 3950
+F 0 "R?" V 4150 3750 50  0000 C CNN
+F 1 "R" V 4200 3950 50  0000 C CNN
+F 2 "" V 4130 3950 50  0001 C CNN
+F 3 "~" H 4200 3950 50  0001 C CNN
+	1    4200 3950
+	0    1    1    0
+$EndComp
+Wire Wire Line
+	4050 3950 3550 3950
+Wire Wire Line
+	4350 3950 4650 3950
+Text Label 4600 7100 2    50   ~ 0
+FPGA_RST
 Wire Bus Line
-	3600 6250 3600 7000
+	3600 6150 3600 7000
 Wire Bus Line
 	2500 6250 2500 7000

Commit message: Add files via upload
Parts:
- added C? (x2): 0.1u, symbol Device:C
- R? (x5): value R -> 100
Connections:
- net GND: now reaches U?.1 (GND), U?.32 (GND)
- net GND: now also C?.1, C?.1
- net +3V3_MCU: now reaches U?.31 (3.3V_VIN)
- net +3V3_MCU: now also C?.2, C?.2
Changed lines of the file:
@@
 $Descr A4 11693 8268
 encoding utf-8
-Sheet 3 4
+Sheet 3 5
 Title ""
 Date ""
@@
 U 1 1 5E83E4D5
 P 5350 3450
-F 0 "U?" H 5350 2161 50  0000 C CNN
-F 1 "Omega2+" H 5350 2070 50  0000 C CNN
+F 0 "U?" H 5500 2400 50  0000 C CNN
+F 1 "Omega2+" H 5750 2400 50  0000 C CNN
 F 2 "Module:Onion_Omega2+" H 5350 1950 50  0001 C CNN
 F 3 "https://docs.onion.io/omega2-docs/omega2p.html" H 2150 2300 50  0001 C CNN
@@
 P 4200 3250
 F 0 "R?" V 4150 3050 50  0000 C CNN
-F 1 "R" V 4200 3250 50  0000 C CNN
+F 1 "100" V 4200 3250 50  0000 C CNN
 F 2 "" V 4130 3250 50  0001 C CNN
 F 3 "~" H 4200 3250 50  0001 C CNN
@@
 P 4200 3350
 F 0 "R?" V 4150 3150 50  0000 C CNN
-F 1 "R" V 4200 3350 50  0000 C CNN
+F 1 "100" V 4200 3350 50  0000 C CNN
 F 2 "" V 4130 3350 50  0001 C CNN
 F 3 "~" H 4200 3350 50  0001 C CNN
@@
 P 4200 3450
 F 0 "R?" V 4150 3250 50  0000 C CNN
-F 1 "R" V 4200 3450 50  0000 C CNN
+F 1 "100" V 4200 3450 50  0000 C CNN
 F 2 "" V 4130 3450 50  0001 C CNN
 F 3 "~" H 4200 3450 50  0001 C CNN
@@
 P 4200 3550
 F 0 "R?" V 4150 3350 50  0000 C CNN
-F 1 "R" V 4200 3550 50  0000 C CNN
+F 1 "100" V 4200 3550 50  0000 C CNN
 F 2 "" V 4130 3550 50  0001 C CNN
 F 3 "~" H 4200 3550 50  0001 C CNN
@@
 P 4200 3950
 F 0 "R?" V 4150 3750 50  0000 C CNN
-F 1 "R" V 4200 3950 50  0000 C CNN
+F 1 "100" V 4200 3950 50  0000 C CNN
 F 2 "" V 4130 3950 50  0001 C CNN
 F 3 "~" H 4200 3950 50  0001 C CNN
@@
 Text Label 4600 7100 2    50   ~ 0
 FPGA_RST
+$Comp
+L Device:C C?
+U 1 1 5EAE2A1D
+P 4800 1700
+AR Path="/5E829221/5EAE2A1D" Ref="C?"  Part="1"
+AR Path="/5E829246/5EAE2A1D" Ref="C?"  Part="1"
+F 0 "C?" V 4750 1500 50  0000 L CNN
+F 1 "0.1u" V 4750 1750 50  0000 L CNN
+F 2 "" H 4838 1550 50  0001 C CNN
+F 3 "~" H 4800 1700 50  0001 C CNN
+	1    4800 1700
+	-1   0    0    1
+$EndComp
+Wire Wire Line
+	4800 1950 4800 1850
+$Comp
+L Device:C C?
+U 1 1 5EAECF58
+P 5050 1700
+AR Path="/5E829221/5EAECF58" Ref="C?"  Part="1"
+AR Path="/5E829246/5EAECF58" Ref="C?"  Part="1"
+F 0 "C?" V 5000 1500 50  0000 L CNN
+F 1 "0.1u" V 5000 1750 50  0000 L CNN
+F 2 "" H 5088 1550 50  0001 C CNN
+F 3 "~" H 5050 1700 50  0001 C CNN
+	1    5050 1700
+	-1   0    0    1
+$EndComp
+Wire Wire Line
+	5050 1850 5050 1950
+Wire Wire Line
+	5050 1950 4950 1950
+Wire Wire Line
+	4800 1550 4800 1350
+Wire Wire Line
+	4800 1350 5050 1350
+Wire Wire Line
+	5250 1350 5250 2250
+Wire Wire Line
+	5050 1550 5050 1350
+Connection ~ 5050 1350
+Wire Wire Line
+	5050 1350 5250 1350
+$Comp
+L power:GND #PWR?
+U 1 1 5EAF103C
+P 4950 2050
+F 0 "#PWR?" H 4950 1800 50  0001 C CNN
+F 1 "GND" H 4955 1877 50  0000 C CNN
+F 2 "" H 4950 2050 50  0001 C CNN
+F 3 "" H 4950 2050 50  0001 C CNN
+	1    4950 2050
+	1    0    0    -1
+$EndComp
+Wire Wire Line
+	4950 2050 4950 1950
+Connection ~ 4950 1950
+Wire Wire Line
+	4950 1950 4800 1950
+Text GLabel 4400 1350 0    50   Input ~ 0
++3V3_MCU
+Wire Wire Line
+	4400 1350 4800 1350
+Connection ~ 4800 1350
+$Comp
+L power:GND #PWR?
+U 1 1 5EAF9EE0
+P 5350 4800
+F 0 "#PWR?" H 5350 4550 50  0001 C CNN
+F 1 "GND" H 5355 4627 50  0000 C CNN
+F 2 "" H 5350 4800 50  0001 C CNN
+F 3 "" H 5350 4800 50  0001 C CNN
+	1    5350 4800
+	1    0    0    -1
+$EndComp
+Wire Wire Line
+	5350 4650 5350 4800
 Wire Bus Line
 	3600 6150 3600 7000

Commit message: Add files via upload
Parts:
- added C?: 33u, symbol Device:C
- added C? (x2): 0.1u, symbol Device:C
- added D?: 1N4733AW, symbol Device:D_Schottky_ALT
- added D?: SP0502BAHT, Package_TO_SOT_SMD:SOT-23, symbol Power_Protection:SP0502BAHT
- added J?: Conn_01x03, symbol Connector_Generic:Conn_01x03
- added J?: USB_A, symbol Connector:USB_A
- added L?: 2A 120 ohm, symbol Device:L
- added R?: 10K, symbol Device:R
- added R? (x2): 33E, symbol Device:R
- added U?: SMS, symbol pulse:SMS
- added U?: SRF2012, symbol SRF:SRF2012
Connections:
- net +3V3_MCU: now also R?.2
- net GND: now also C?.2, C?.2, C?.2, D?.2 (A), D?.3 (A), J?.1 (Pin_1), J?.4 (GND), J?.5 (Shield), U?.3, U?.4
- net RST: now reaches U?.26 (FW_RST/38)
- net RST: now also C?.1, R?.1, U?.1, U?.2
- net at U?.27 (SER0_TX/12): now also R?.2
- net at U?.28 (SER0_RX/13): now also R?.2
- net USB_D-: now reaches U?.29 (USB_D-)
- net USB_D-: now also U?.3
- net USB_D+: now reaches U?.30 (USB_D+)
- net USB_D+: now also U?.2
- new net: C?.1, C?.1, D?.1 (K), J?.1 (VBUS), L?.1
- new net: J?.2 (Pin_2), R?.1
- new net: J?.3 (Pin_3), R?.1
- new net: D?.1 (K), J?.2 (D-), U?.4
- new net: D?.2 (K), J?.3 (D+), U?.1
- new net +5V: L?.2
Other:
- moved on the sheet: C?, R?, U?

Commit message: Add files via upload
Parts:
- gave numbers to parts that had none: 21
Changed lines of the file:
@@
 $EndDescr
 $Comp
-L MCU_Module:Omega2+ U?
+L MCU_Module:Omega2+ U6
 U 1 1 5E83E4D5
 P 3750 3000
-F 0 "U?" H 3900 1950 50  0000 C CNN
+F 0 "U6" H 3900 1950 50  0000 C CNN
 F 1 "Omega2+" H 4150 1950 50  0000 C CNN
 F 2 "Module:Onion_Omega2+" H 3750 1500 50  0001 C CNN
@@
 	4450 3100 4750 3100
 $Comp
-L Device:R R?
+L Device:R R46
 U 1 1 5E8EEB33
 P 2600 2800
-F 0 "R?" V 2550 2600 50  0000 C CNN
+F 0 "R46" V 2550 2600 50  0000 C CNN
 F 1 "100" V 2600 2800 50  0000 C CNN
 F 2 "" V 2530 2800 50  0001 C CNN
@@
 $EndComp
 $Comp
-L Device:R R?
+L Device:R R47
 U 1 1 5E8F0E74
 P 2600 2900
-F 0 "R?" V 2550 2700 50  0000 C CNN
+F 0 "R47" V 2550 2700 50  0000 C CNN
 F 1 "100" V 2600 2900 50  0000 C CNN
 F 2 "" V 2530 2900 50  0001 C CNN
@@
 $EndComp
 $Comp
-L Device:R R?
+L Device:R R48
 U 1 1 5E8F157B
 P 2600 3000
-F 0 "R?" V 2550 2800 50  0000 C CNN
+F 0 "R48" V 2550 2800 50  0000 C CNN
 F 1 "100" V 2600 3000 50  0000 C CNN
 F 2 "" V 2530 3000 50  0001 C CNN
@@
 $EndComp
 $Comp
-L Device:R R?
+L Device:R R49
 U 1 1 5E8F1C79
 P 2600 3100
-F 0 "R?" V 2550 2900 50  0000 C CNN
+F 0 "R49" V 2550 2900 50  0000 C CNN
 F 1 "100" V 2600 3100 50  0000 C CNN
 F 2 "" V 2530 3100 50  0001 C CNN
@@
 FPGA_RST
 $Comp
-L Device:R R?
+L Device:R R50
 U 1 1 5E87BB84
 P 2600 3500
-F 0 "R?" V 2550 3300 50  0000 C CNN
+F 0 "R50" V 2550 3300 50  0000 C CNN
 F 1 "100" V 2600 3500 50  0000 C CNN
 F 2 "" V 2530 3500 50  0001 C CNN
@@
 P 3200 1250
 AR Path="/5E829221/5EAE2A1D" Ref="C?"  Part="1"
-AR Path="/5E829246/5EAE2A1D" Ref="C?"  Part="1"
-F 0 "C?" V 3150 1050 50  0000 L CNN
+AR Path="/5E829246/5EAE2A1D" Ref="C20"  Part="1"
+F 0 "C20" V 3150 1050 50  0000 L CNN
 F 1 "0.1u" V 3150 1300 50  0000 L CNN
 F 2 "" H 3238 1100 50  0001 C CNN
@@
 P 3450 1250
 AR Path="/5E829221/5EAECF58" Ref="C?"  Part="1"
-AR Path="/5E829246/5EAECF58" Ref="C?"  Part="1"
-F 0 "C?" V 3400 1050 50  0000 L CNN
+AR Path="/5E829246/5EAECF58" Ref="C21"  Part="1"
+F 0 "C21" V 3400 1050 50  0000 L CNN
 F 1 "0.1u" V 3400 1300 50  0000 L CNN
 F 2 "" H 3488 1100 50  0001 C CNN
@@
 	3450 900  3650 900
 $Comp
-L power:GND #PWR?
+L power:GND #PWR023
 U 1 1 5EAF103C
 P 3350 1600
-F 0 "#PWR?" H 3350 1350 50  0001 C CNN
+F 0 "#PWR023" H 3350 1350 50  0001 C CNN
 F 1 "GND" H 3355 1427 50  0000 C CNN
 F 2 "" H 3350 1600 50  0001 C CNN
@@
 Connection ~ 3200 900
 $Comp
-L power:GND #PWR?
+L power:GND #PWR024
 U 1 1 5EAF9EE0
 P 3750 4350
-F 0 "#PWR?" H 3750 4100 50  0001 C CNN
+F 0 "#PWR024" H 3750 4100 50  0001 C CNN
 F 1 "GND" H 3755 4177 50  0000 C CNN
 F 2 "" H 3750 4350 50  0001 C CNN
@@
 	3750 4200 3750 4350
 $Comp
-L Connector:USB_A J?
+L Connector:USB_A J4
 U 1 1 5EC8AFBF
 P 8250 1850
-F 0 "J?" H 8307 2317 50  0000 C CNN
+F 0 "J4" H 8307 2317 50  0000 C CNN
 F 1 "USB_A" H 8307 2226 50  0000 C CNN
 F 2 "" H 8400 1800 50  0001 C CNN
@@
 $EndComp
 $Comp
-L Power_Protection:SP0502BAHT D?
+L Power_Protection:SP0502BAHT D5
 U 1 1 5EC8E69C
 P 9100 2250
-F 0 "D?" H 9305 2296 50  0000 L CNN
+F 0 "D5" H 9305 2296 50  0000 L CNN
 F 1 "SP0502BAHT" H 9305 2205 50  0000 L CNN
 F 2 "Package_TO_SOT_SMD:SOT-23" H 9325 2200 50  0001 L CNN
@@
 $EndComp
 $Comp
-L SRF:SRF2012 U?
+L SRF:SRF2012 U8
 U 1 1 5EC9479E
 P 9600 1900
-F 0 "U?" H 9600 2175 50  0000 C CNN
+F 0 "U8" H 9600 2175 50  0000 C CNN
 F 1 "SRF2012" H 9600 2084 50  0000 C CNN
 F 2 "" H 9600 2150 50  0001 C CNN
@@
 	9000 1950 8550 1950
 $Comp
-L power:GND #PWR?
+L power:GND #PWR026
 U 1 1 5EC9B689
 P 8150 2400
-F 0 "#PWR?" H 8150 2150 50  0001 C CNN
+F 0 "#PWR026" H 8150 2150 50  0001 C CNN
 F 1 "GND" H 8155 2227 50  0000 C CNN
 F 2 "" H 8150 2400 50  0001 C CNN
@@
 $EndComp
 $Comp
-L power:GND #PWR?
+L power:GND #PWR027
 U 1 1 5EC9BB41
 P 9100 2550
-F 0 "#PWR?" H 9100 2300 50  0001 C CNN
+F 0 "#PWR027" H 9100 2300 50  0001 C CNN
 F 1 "GND" H 9105 2377 50  0000 C CNN
 F 2 "" H 9100 2550 50  0001 C CNN
@@
 	8150 2350 8150 2250
 $Comp
-L Device:D_Schottky_ALT D?
+L Device:D_Schottky_ALT D4
 U 1 1 5E953A1A
 P 8750 1150
-F 0 "D?" V 8704 1229 50  0000 L CNN
+F 0 "D4" V 8704 1229 50  0000 L CNN
 F 1 "1N4733AW" V 8795 1229 50  0000 L CNN
 F 2 "" H 8750 1150 50  0001 C CNN
@@
 $EndComp
 $Comp
-L Device:C C?
+L Device:C C22
 U 1 1 5E953DE8
 P 9600 1150
-F 0 "C?" H 9715 1196 50  0000 L CNN
+F 0 "C22" H 9715 1196 50  0000 L CNN
 F 1 "33u" H 9715 1105 50  0000 L CNN
 F 2 "" H 9638 1000 50  0001 C CNN
@@
 $EndComp
 $Comp
-L Device:C C?
+L Device:C C23
 U 1 1 5E954221
 P 9950 1150
-F 0 "C?" H 10065 1196 50  0000 L CNN
+F 0 "C23" H 10065 1196 50  0000 L CNN
 F 1 "0.1u" H 10065 1105 50  0000 L CNN
 F 2 "" H 9988 1000 50  0001 C CNN
@@
 $EndComp
 $Comp
-L Device:L L?
+L Device:L L1
 U 1 1 5E9548AA
 P 10300 900
-F 0 "L?" V 10490 900 50  0000 C CNN
+F 0 "L1" V 10490 900 50  0000 C CNN
 F 1 "2A 120 ohm" V 10399 900 50  0000 C CNN
 F 2 "" H 10300 900 50  0001 C CNN
@@
 Connection ~ 8750 900
 $Comp
-L power:GND #PWR?
+L power:GND #PWR028
 U 1 1 5E9666D3
 P 9200 1450
-F 0 "#PWR?" H 9200 1200 50  0001 C CNN
+F 0 "#PWR028" H 9200 1200 50  0001 C CNN
 F 1 "GND" H 9205 1277 50  0000 C CNN
 F 2 "" H 9200 1450 50  0001 C CNN
@@
 AR Path="/5E926AEA/5E9A2EDA" Ref="R?"  Part="1"
 AR Path="/5E829221/5E9A2EDA" Ref="R?"  Part="1"
-AR Path="/5E829246/5E9A2EDA" Ref="R?"  Part="1"
-F 0 "R?" V 8950 3650 50  0000 L CNN
+AR Path="/5E829246/5E9A2EDA" Ref="R53"  Part="1"
+F 0 "R53" V 8950 3650 50  0000 L CNN
 F 1 "10K" V 8900 3500 50  0000 L CNN
 F 2 "" V 8830 3550 50  0001 C CNN
@@
 	8900 3700 8900 3750
 $Comp
-L pulse:SMS U?
+L pulse:SMS U7
 U 1 1 5E9A2EE3
 P 9450 4150
-F 0 "U?" H 9450 4425 50  0000 C CNN
+F 0 "U7" H 9450 4425 50  0000 C CNN
 F 1 "SMS" H 9450 4334 50  0000 C CNN
 F 2 "" H 9850 4350 50  0001 C CNN
@@
 	9700 3750 10050 3750
 $Comp
-L power:GND #PWR?
+L power:GND #PWR029
 U 1 1 5E9A2EEE
 P 9200 4400
-F 0 "#PWR?" H 9200 4150 50  0001 C CNN
+F 0 "#PWR029" H 9200 4150 50  0001 C CNN
 F 1 "GND" H 9205 4227 50  0000 C CNN
 F 2 "" H 9200 4400 50  0001 C CNN
@@
 $EndComp
 $Comp
-L power:GND #PWR?
+L power:GND #PWR030
 U 1 1 5E9A2EF4
 P 9700 4400
-F 0 "#PWR?" H 9700 4150 50  0001 C CNN
+F 0 "#PWR030" H 9700 4150 50  0001 C CNN
 F 1 "GND" H 9705 4227 50  0000 C CNN
 F 2 "" H 9700 4400 50  0001 C CNN
@@
 	9200 4250 9200 4400
 $Comp
-L power:GND #PWR?
+L power:GND #PWR031
 U 1 1 5E9A2EFC
 P 10050 4250
-F 0 "#PWR?" H 10050 4000 50  0001 C CNN
+F 0 "#PWR031" H 10050 4000 50  0001 C CNN
 F 1 "GND" H 10055 4077 50  0000 C CNN
 F 2 "" H 10050 4250 50  0001 C CNN
@@
 	10050 4150 10050 4250
 $Comp
-L Device:C C?
+L Device:C C24
 U 1 1 5E9A2F05
 P 10050 4000
-F 0 "C?" H 10165 4046 50  0000 L CNN
+F 0 "C24" H 10165 4046 50  0000 L CNN
 F 1 "0.1u" H 10165 3955 50  0000 L CNN
 F 2 "" H 10088 3850 50  0001 C CNN
@@
 	7900 4800 7900 2850
 $Comp
-L Connector_Generic:Conn_01x03 J?
+L Connector_Generic:Conn_01x03 J3
 U 1 1 5E9D5094
 P 5500 2700
-F 0 "J?" H 5580 2742 50  0000 L CNN
+F 0 "J3" H 5580 2742 50  0000 L CNN
 F 1 "Conn_01x03" H 5580 2651 50  0000 L CNN
 F 2 "" H 5500 2700 50  0001 C CNN
@@
 $EndComp
 $Comp
-L Device:R R?
+L Device:R R51
 U 1 1 5E9D7503
 P 4950 2700
-F 0 "R?" V 4900 2550 50  0000 C CNN
+F 0 "R51" V 4900 2500 50  0000 C CNN
 F 1 "33E" V 4950 2700 50  0000 C CNN
 F 2 "" V 4880 2700 50  0001 C CNN
@@
 $EndComp
 $Comp
-L Device:R R?
+L Device:R R52
 U 1 1 5E9DF0D8
 P 4950 2800
-F 0 "R?" V 4900 2650 50  0000 C CNN
+F 0 "R52" V 4900 2600 50  0000 C CNN
 F 1 "33E" V 4950 2800 50  0000 C CNN
 F 2 "" V 4880 2800 50  0001 C CNN
@@
 	4450 2700 4800 2700
 $Comp
-L power:GND #PWR?
+L power:GND #PWR025
 U 1 1 5E9E9A66
 P 5250 2500
-F 0 "#PWR?" H 5250 2250 50  0001 C CNN
+F 0 "#PWR025" H 5250 2250 50  0001 C CNN
 F 1 "GND" H 5255 2327 50  0000 C CNN
 F 2 "" H 5250 2500 50  0001 C CNN

Commit message: Add files via upload
Parts:
- C20, C21, C22, C23, C24: footprint (none) -> Capacitor_SMD:C_0805_2012Metric_Pad1.15x1.40mm_HandSolder
- J3: footprint (none) -> Connector_PinHeader_2.54mm:PinHeader_1x03_P2.54mm_Vertical
- R46, R47, R48, R49, R50, R53: footprint (none) -> Resistor_SMD:R_0603_1608Metric_Pad1.05x0.95mm_HandSolder
Changed lines of the file:
@@
 F 0 "R46" V 2550 2600 50  0000 C CNN
 F 1 "100" V 2600 2800 50  0000 C CNN
-F 2 "" V 2530 2800 50  0001 C CNN
+F 2 "Resistor_SMD:R_0603_1608Metric_Pad1.05x0.95mm_HandSolder" V 2530 2800 50  0001 C CNN
 F 3 "~" H 2600 2800 50  0001 C CNN
 	1    2600 2800
@@
 F 0 "R47" V 2550 2700 50  0000 C CNN
 F 1 "100" V 2600 2900 50  0000 C CNN
-F 2 "" V 2530 2900 50  0001 C CNN
+F 2 "Resistor_SMD:R_0603_1608Metric_Pad1.05x0.95mm_HandSolder" V 2530 2900 50  0001 C CNN
 F 3 "~" H 2600 2900 50  0001 C CNN
 	1    2600 2900
@@
 F 0 "R48" V 2550 2800 50  0000 C CNN
 F 1 "100" V 2600 3000 50  0000 C CNN
-F 2 "" V 2530 3000 50  0001 C CNN
+F 2 "Resistor_SMD:R_0603_1608Metric_Pad1.05x0.95mm_HandSolder" V 2530 3000 50  0001 C CNN
 F 3 "~" H 2600 3000 50  0001 C CNN
 	1    2600 3000
@@
 F 0 "R49" V 2550 2900 50  0000 C CNN
 F 1 "100" V 2600 3100 50  0000 C CNN
-F 2 "" V 2530 3100 50  0001 C CNN
+F 2 "Resistor_SMD:R_0603_1608Metric_Pad1.05x0.95mm_HandSolder" V 2530 3100 50  0001 C CNN
 F 3 "~" H 2600 3100 50  0001 C CNN
 	1    2600 3100
@@
 F 0 "R50" V 2550 3300 50  0000 C CNN
 F 1 "100" V 2600 3500 50  0000 C CNN
-F 2 "" V 2530 3500 50  0001 C CNN
+F 2 "Resistor_SMD:R_0603_1608Metric_Pad1.05x0.95mm_HandSolder" V 2530 3500 50  0001 C CNN
 F 3 "~" H 2600 3500 50  0001 C CNN
 	1    2600 3500
@@
 F 0 "C20" V 3150 1050 50  0000 L CNN
 F 1 "0.1u" V 3150 1300 50  0000 L CNN
-F 2 "" H 3238 1100 50  0001 C CNN
+F 2 "Capacitor_SMD:C_0805_2012Metric_Pad1.15x1.40mm_HandSolder" H 3238 1100 50  0001 C CNN
 F 3 "~" H 3200 1250 50  0001 C CNN
 	1    3200 1250
@@
 F 0 "C21" V 3400 1050 50  0000 L CNN
 F 1 "0.1u" V 3400 1300 50  0000 L CNN
-F 2 "" H 3488 1100 50  0001 C CNN
+F 2 "Capacitor_SMD:C_0805_2012Metric_Pad1.15x1.40mm_HandSolder" H 3488 1100 50  0001 C CNN
 F 3 "~" H 3450 1250 50  0001 C CNN
 	1    3450 1250
@@
 F 0 "C22" H 9715 1196 50  0000 L CNN
 F 1 "33u" H 9715 1105 50  0000 L CNN
-F 2 "" H 9638 1000 50  0001 C CNN
+F 2 "Capacitor_SMD:C_0805_2012Metric_Pad1.15x1.40mm_HandSolder" H 9638 1000 50  0001 C CNN
 F 3 "~" H 9600 1150 50  0001 C CNN
 	1    9600 1150
@@
 F 0 "C23" H 10065 1196 50  0000 L CNN
 F 1 "0.1u" H 10065 1105 50  0000 L CNN
-F 2 "" H 9988 1000 50  0001 C CNN
+F 2 "Capacitor_SMD:C_0805_2012Metric_Pad1.15x1.40mm_HandSolder" H 9988 1000 50  0001 C CNN
 F 3 "~" H 9950 1150 50  0001 C CNN
 	1    9950 1150
@@
 F 0 "R53" V 8950 3650 50  0000 L CNN
 F 1 "10K" V 8900 3500 50  0000 L CNN
-F 2 "" V 8830 3550 50  0001 C CNN
+F 2 "Resistor_SMD:R_0603_1608Metric_Pad1.05x0.95mm_HandSolder" V 8830 3550 50  0001 C CNN
 F 3 "~" H 8900 3550 50  0001 C CNN
 	1    8900 3550
@@
 F 0 "C24" H 10165 4046 50  0000 L CNN
 F 1 "0.1u" H 10165 3955 50  0000 L CNN
-F 2 "" H 10088 3850 50  0001 C CNN
+F 2 "Capacitor_SMD:C_0805_2012Metric_Pad1.15x1.40mm_HandSolder" H 10088 3850 50  0001 C CNN
 F 3 "~" H 10050 4000 50  0001 C CNN
 	1    10050 4000
@@
 F 0 "J3" H 5580 2742 50  0000 L CNN
 F 1 "Conn_01x03" H 5580 2651 50  0000 L CNN
-F 2 "" H 5500 2700 50  0001 C CNN
+F 2 "Connector_PinHeader_2.54mm:PinHeader_1x03_P2.54mm_Vertical" H 5500 2700 50  0001 C CNN
 F 3 "~" H 5500 2700 50  0001 C CNN
 	1    5500 2700

Commit message: Add files via upload
Parts:
- D4: footprint (none) -> Diode_SMD:D_SOD-123
- J4: footprint (none) -> Connector_USB:USB_A_Wuerth_61400826021_Horizontal_Stacked
- L1: footprint (none) -> Inductor_SMD:L_0805_2012Metric_Pad1.15x1.40mm_HandSolder
- U7: footprint (none) -> AICE:SMS_BUTTON
- U8: footprint (none) -> AICE:SRF2012
Changed lines of the file:
@@
 F 0 "J4" H 8307 2317 50  0000 C CNN
 F 1 "USB_A" H 8307 2226 50  0000 C CNN
-F 2 "" H 8400 1800 50  0001 C CNN
+F 2 "Connector_USB:USB_A_Wuerth_61400826021_Horizontal_Stacked" H 8400 1800 50  0001 C CNN
 F 3 " ~" H 8400 1800 50  0001 C CNN
 	1    8250 1850
@@
 F 0 "U8" H 9600 2175 50  0000 C CNN
 F 1 "SRF2012" H 9600 2084 50  0000 C CNN
-F 2 "" H 9600 2150 50  0001 C CNN
+F 2 "AICE:SRF2012" H 9600 2150 50  0001 C CNN
 F 3 "" H 9600 2150 50  0001 C CNN
 	1    9600 1900
@@
 F 0 "D4" V 8704 1229 50  0000 L CNN
 F 1 "1N4733AW" V 8795 1229 50  0000 L CNN
-F 2 "" H 8750 1150 50  0001 C CNN
+F 2 "Diode_SMD:D_SOD-123" H 8750 1150 50  0001 C CNN
 F 3 "~" H 8750 1150 50  0001 C CNN
 	1    8750 1150
@@
 F 0 "L1" V 10490 900 50  0000 C CNN
 F 1 "2A 120 ohm" V 10399 900 50  0000 C CNN
-F 2 "" H 10300 900 50  0001 C CNN
+F 2 "Inductor_SMD:L_0805_2012Metric_Pad1.15x1.40mm_HandSolder" H 10300 900 50  0001 C CNN
 F 3 "~" H 10300 900 50  0001 C CNN
 	1    10300 900
@@
 F 0 "U7" H 9450 4425 50  0000 C CNN
 F 1 "SMS" H 9450 4334 50  0000 C CNN
-F 2 "" H 9850 4350 50  0001 C CNN
+F 2 "AICE:SMS_BUTTON" H 9850 4350 50  0001 C CNN
 F 3 "" H 9850 4350 50  0001 C CNN
 	1    9450 4150
