File: AICE/omega.sch (KiCad schematic (older format))
At the start: 20 parts, among them J3 Conn_01x03, J4 USB_A, U6 Omega2+, U7 SMS, U8 SRF2012

Commit message: Add files via upload
Parts:
- C22: footprint Capacitor_SMD:C_0805_2012Metric -> Capacitor_THT:CP_Radial_D5.0mm_P2.00mm
Changed lines of the file:
@@
 F 0 "C22" H 9715 1196 50  0000 L CNN
 F 1 "33u" H 9715 1105 50  0000 L CNN
-F 2 "Capacitor_SMD:C_0805_2012Metric" H 9638 1000 50  0001 C CNN
+F 2 "Capacitor_THT:CP_Radial_D5.0mm_P2.00mm" H 9638 1000 50  0001 C CNN
 F 3 "~" H 9600 1150 50  0001 C CNN
 	1    9600 1150

Commit message: Add files via upload
Parts:
- added R7: 10K, Resistor_SMD:R_0603_1608Metric, symbol Device:R
Connections:
- net GND: now also R7.1
- net OmSPI2: now also R7.2
Changed lines of the file:
@@
 SPI_MISO
-Wire Wire Line
-	1950 2900 2450 2900
-Wire Wire Line
-	2450 2800 1950 2800
 Wire Wire Line
 	1950 3000 2450 3000
@@
 NoConn ~ 3050 2400
 NoConn ~ 3050 3600
+$Comp
+L Device:R R?
+U 1 1 5EC8FF55
+P 1650 3050
+AR Path="/5E926AEA/5EC8FF55" Ref="R?"  Part="1"
+AR Path="/5E829221/5EC8FF55" Ref="R?"  Part="1"
+AR Path="/5E829246/5EC8FF55" Ref="R7"  Part="1"
+F 0 "R7" V 1700 3150 50  0000 L CNN
+F 1 "10K" V 1650 3000 50  0000 L CNN
+F 2 "Resistor_SMD:R_0603_1608Metric" V 1580 3050 50  0001 C CNN
+F 3 "~" H 1650 3050 50  0001 C CNN
+	1    1650 3050
+	-1   0    0    1
+$EndComp
+$Comp
+L power:GND #PWR038
+U 1 1 5EC950AE
+P 1650 3250
+F 0 "#PWR038" H 1650 3000 50  0001 C CNN
+F 1 "GND" H 1655 3077 50  0000 C CNN
+F 2 "" H 1650 3250 50  0001 C CNN
+F 3 "" H 1650 3250 50  0001 C CNN
+	1    1650 3250
+	1    0    0    -1
+$EndComp
+Wire Wire Line
+	1650 3250 1650 3200
+Wire Wire Line
+	2450 2800 1950 2800
+Wire Wire Line
+	1650 2900 2450 2900
 Wire Bus Line
 	9900 5050 9900 5900
