File: AICE/power.sch (KiCad schematic (older format))
At the start: 58 parts, among them J8 USB_B_Micro, U13 ZLDO1117G33TA, U14 XC6206P122MR, U15 ZLDO1117G33TA, U16 ZLDO1117G18TA, U17 XC6206P282MR, U18 XC6206P152MR

Commit message: Add files via upload
Changed lines of the file:
@@
 Connection ~ 7700 2800
-Wire Wire Line
-	7700 2800 7500 2800
 Wire Wire Line
 	7700 3200 7700 3350
@@
 Wire Wire Line
 	9050 2800 9300 2800
-Text GLabel 7500 2800 0    50   Input ~ 0
-+5V
 Text GLabel 9500 2800 2    50   Input ~ 0
 +2V8_MCU
@@
 Wire Wire Line
 	1650 3950 1850 3950
+Text GLabel 7300 2800 0    50   Input ~ 0
++5V
+Wire Wire Line
+	7300 2800 7700 2800
 $EndSCHEMATC

Commit message: Add files via upload
Parts:
- removed D11: BLU, LED_SMD:LED_0603_1608Metric, symbol Device:LED_ALT
- removed D12, D9: GRN, LED_SMD:LED_0603_1608Metric, symbol Device:LED_ALT
- removed D13: YLL, LED_SMD:LED_0603_1608Metric, symbol Device:LED_ALT
- removed R100, R101, R97, R99: 2k2, Resistor_SMD:R_0603_1608Metric, symbol Device:R
Changed lines of the file:
@@
 Wire Wire Line
 	5550 1950 5550 2050
-$Comp
-L Device:LED_ALT D9
-U 1 1 5E9AA529
-P 6150 1350
-F 0 "D9" H 6050 1400 50  0000 R CNN
-F 1 "GRN" H 6350 1400 50  0000 R CNN
-F 2 "LED_SMD:LED_0603_1608Metric" H 6150 1350 50  0001 C CNN
-F 3 "~" H 6150 1350 50  0001 C CNN
-	1    6150 1350
-	0    -1   -1   0
-$EndComp
-$Comp
-L Device:R R97
-U 1 1 5E9AA52F
-P 6150 1800
-F 0 "R97" V 6100 1550 50  0000 L CNN
-F 1 "2k2" V 6150 1700 50  0000 L CNN
-F 2 "Resistor_SMD:R_0603_1608Metric" V 6080 1800 50  0001 C CNN
-F 3 "~" H 6150 1800 50  0001 C CNN
-	1    6150 1800
-	1    0    0    -1
-$EndComp
-Wire Wire Line
-	6150 1500 6150 1650
-Wire Wire Line
-	6150 1950 6150 2050
 Text GLabel 5550 1000 0    50   Input ~ 0
 +3V3_FPGA
-Text GLabel 6150 1000 0    50   Input ~ 0
-+1V2_FPGA
 $Comp
 L Device:LED_ALT D10
@@
 	6850 1950 6850 2050
 $Comp
-L Device:LED_ALT D11
-U 1 1 5E9C6197
-P 7450 1350
-F 0 "D11" H 7350 1400 50  0000 R CNN
-F 1 "BLU" H 7650 1400 50  0000 R CNN
-F 2 "LED_SMD:LED_0603_1608Metric" H 7450 1350 50  0001 C CNN
-F 3 "~" H 7450 1350 50  0001 C CNN
-	1    7450 1350
-	0    -1   -1   0
-$EndComp
-$Comp
-L Device:R R99
-U 1 1 5E9C619D
-P 7450 1800
-F 0 "R99" V 7400 1550 50  0000 L CNN
-F 1 "2k2" V 7450 1700 50  0000 L CNN
-F 2 "Resistor_SMD:R_0603_1608Metric" V 7380 1800 50  0001 C CNN
-F 3 "~" H 7450 1800 50  0001 C CNN
-	1    7450 1800
-	1    0    0    -1
-$EndComp
-Wire Wire Line
-	7450 1500 7450 1650
-Wire Wire Line
-	7450 1950 7450 2050
-$Comp
 L power:GND #PWR065
 U 1 1 5E9CF9D2
@@
 $EndComp
 $Comp
-L power:GND #PWR066
-U 1 1 5E9D0CD1
-P 6150 2050
-F 0 "#PWR066" H 6150 1800 50  0001 C CNN
-F 1 "GND" H 6155 1877 50  0000 C CNN
-F 2 "" H 6150 2050 50  0001 C CNN
-F 3 "" H 6150 2050 50  0001 C CNN
-	1    6150 2050
-	1    0    0    -1
-$EndComp
-$Comp
 L power:GND #PWR067
 U 1 1 5E9D0F98
@@
 	1    0    0    -1
 $EndComp
-$Comp
-L power:GND #PWR068
-U 1 1 5E9D1282
-P 7450 2050
-F 0 "#PWR068" H 7450 1800 50  0001 C CNN
-F 1 "GND" H 7455 1877 50  0000 C CNN
-F 2 "" H 7450 2050 50  0001 C CNN
-F 3 "" H 7450 2050 50  0001 C CNN
-	1    7450 2050
-	1    0    0    -1
-$EndComp
 Text GLabel 6850 1000 0    50   Input ~ 0
 +3V3_MCU
-Text GLabel 7450 1000 0    50   Input ~ 0
-+1V8_MCU
-Wire Wire Line
-	7450 1000 7450 1200
 Wire Wire Line
 	6850 1000 6850 1200
-Wire Wire Line
-	6150 1000 6150 1200
 Wire Wire Line
 	5550 1000 5550 1200
@@
 Wire Notes Line
 	4050 2350 10050 2350
-$Comp
-L Device:LED_ALT D12
-U 1 1 5EC27737
-P 8100 1350
-F 0 "D12" H 8000 1400 50  0000 R CNN
-F 1 "GRN" H 8300 1400 50  0000 R CNN
-F 2 "LED_SMD:LED_0603_1608Metric" H 8100 1350 50  0001 C CNN
-F 3 "~" H 8100 1350 50  0001 C CNN
-	1    8100 1350
-	0    -1   -1   0
-$EndComp
-$Comp
-L Device:R R100
-U 1 1 5EC2773D
-P 8100 1800
-F 0 "R100" V 8050 1500 50  0000 L CNN
-F 1 "2k2" V 8100 1700 50  0000 L CNN
-F 2 "Resistor_SMD:R_0603_1608Metric" V 8030 1800 50  0001 C CNN
-F 3 "~" H 8100 1800 50  0001 C CNN
-	1    8100 1800
-	1    0    0    -1
-$EndComp
-Wire Wire Line
-	8100 1500 8100 1650
-Wire Wire Line
-	8100 1950 8100 2050
-$Comp
-L power:GND #PWR069
-U 1 1 5EC27745
-P 8100 2050
-F 0 "#PWR069" H 8100 1800 50  0001 C CNN
-F 1 "GND" H 8105 1877 50  0000 C CNN
-F 2 "" H 8100 2050 50  0001 C CNN
-F 3 "" H 8100 2050 50  0001 C CNN
-	1    8100 2050
-	1    0    0    -1
-$EndComp
-Text GLabel 8100 1000 0    50   Input ~ 0
-+1V5_MCU
-Wire Wire Line
-	8100 1000 8100 1200
-$Comp
-L Device:LED_ALT D13
-U 1 1 5EC2D8AD
-P 8750 1350
-F 0 "D13" H 8650 1400 50  0000 R CNN
-F 1 "YLL" H 8950 1400 50  0000 R CNN
-F 2 "LED_SMD:LED_0603_1608Metric" H 8750 1350 50  0001 C CNN
-F 3 "~" H 8750 1350 50  0001 C CNN
-	1    8750 1350
-	0    -1   -1   0
-$EndComp
-$Comp
-L Device:R R101
-U 1 1 5EC2D8B3
-P 8750 1800
-F 0 "R101" V 8700 1500 50  0000 L CNN
-F 1 "2k2" V 8750 1700 50  0000 L CNN
-F 2 "Resistor_SMD:R_0603_1608Metric" V 8680 1800 50  0001 C CNN
-F 3 "~" H 8750 1800 50  0001 C CNN
-	1    8750 1800
-	1    0    0    -1
-$EndComp
-Wire Wire Line
-	8750 1500 8750 1650
-Wire Wire Line
-	8750 1950 8750 2050
-$Comp
-L power:GND #PWR072
-U 1 1 5EC2D8BB
-P 8750 2050
-F 0 "#PWR072" H 8750 1800 50  0001 C CNN
-F 1 "GND" H 8755 1877 50  0000 C CNN
-F 2 "" H 8750 2050 50  0001 C CNN
-F 3 "" H 8750 2050 50  0001 C CNN
-	1    8750 2050
-	1    0    0    -1
-$EndComp
-Text GLabel 8750 1000 0    50   Input ~ 0
-+2V8_MCU
-Wire Wire Line
-	8750 1000 8750 1200
 Wire Notes Line
 	10050 700  10050 2300
