File: AICE/AICE.kicad_pcb (KiCad board)
At the start: 2 copper layers, 150 parts, among them J1 Conn_02x10_Odd_Even, J2 Conn_02x10_Odd_Even, J3 Conn_01x03, J4 USB_A, J5 Conn_02x11_Odd_Even, J6 Conn_02x11_Odd_Even, J7 Micro_SD_Card, J8 USB_B_Micro, Q1 S8550, U1 ICE40UP5K-SG48ITR, U10 SMS, U11 DVP_PORT, U12 SMS, U13 ZLDO1117G33TA, U14 ZLDO1117G12TA, U15 ZLDO1117G33TA, U16 ZLDO1117G18TA, U17 XC6206P282MR, U18 XC6206P152MR, U2 ASFLMB-24.00MHZ-LC-T, U3 SMS, U4 W25Q, U5 HX711, U6 Omega2+, U7 SMS, U8 SRF2012, U9 M1&M1W

Commit message: Add files via upload
Parts:
- added C61: 0.1u, Capacitor_SMD:C_0603_1608Metric_Pad1.05x0.95mm_HandSolder, F.Cu at (79.1, 61.0)
- C19, C24, C26, L4, L5, L6, L7, R4, R53, R90: moved to B.Cu
- moved D1 330.0 mm to (66.2, 87.3), turned to 270 degrees
- moved C3 329.5 mm to (68.7, 88.3), turned to 0 degrees
- moved R37 325.3 mm to (40.2, 88.2), turned to 180 degrees
- moved R102 323.1 mm to (40.2, 90.4), turned to 180 degrees
- moved D3 322.8 mm to (46.2, 90.4), turned to 0 degrees
- moved C19 315.1 mm to (48.8, 75.7), turned to 270 degrees
- moved R103 313.5 mm to (40.2, 92.5), turned to 180 degrees
- moved R5 306.8 mm to (53.7, 63.8), turned to 180 degrees
- moved R6 306.6 mm to (53.7, 62.3), turned to 180 degrees
- moved R4 306.3 mm to (50.4, 75.7), turned to 270 degrees
- moved U3 299.3 mm to (42.3, 75.5)
- moved J3 297.6 mm to (106.7, 139.7)
- moved C17 294.1 mm to (56.3, 63.2)
- moved C22 276.8 mm to (118.5, 126.9)
- moved C23 276.8 mm to (118.4, 123.8)
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
Commit message: Add files via upload
Parts:
- moved J1 60.5 mm to (38.1, 101.3), turned to 180 degrees
- moved R89 54.0 mm to (80.7, 61.4), turned to 90 degrees
- moved R104 53.8 mm to (78.7, 61.4), turned to 90 degrees
- moved R105 53.8 mm to (76.7, 61.4), turned to 90 degrees
- moved U7 47.3 mm to (86.9, 45.3), turned to 0 degrees
- moved D6 44.9 mm to (78.7, 67.7), turned to 270 degrees
- moved U12 43.6 mm to (79.8, 45.5), turned to 0 degrees
- moved R2 43.1 mm to (65.0, 66.1), turned to 270 degrees
- moved U3 42.5 mm to (72.3, 45.4), turned to 0 degrees
- moved R37 42.3 mm to (73.1, 61.5), turned to 90 degrees
- moved R102 42.1 mm to (70.9, 61.5), turned to 90 degrees
- moved R103 42.1 mm to (68.8, 61.6), turned to 90 degrees
- moved U10 40.6 mm to (67.1, 47.2), turned to 180 degrees
- moved C24 39.2 mm to (86.9, 51.8), turned to 180 degrees
- moved J2 38.5 mm to (35.6, 50.5), turned to 0 degrees
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Connections:
- J1 pad 19: /iCE40/SDA -> /iCE40/IO15
- J1 pad 20: /iCE40/SCK -> /iCE40/IO16
- J2 pad 10: /iCE40/IO20 -> /iCE40/E+
- J2 pad 11: /iCE40/IO21 -> /iCE40/IO17
- J2 pad 12: /iCE40/IO22 -> /iCE40/S-
- J2 pad 13: /iCE40/IO23 -> /iCE40/IO19
- J2 pad 14: /iCE40/IO24 -> /iCE40/IO18
- J2 pad 15: /iCE40/IO25 -> /iCE40/IO21
- J2 pad 16: /iCE40/E+ -> /iCE40/IO20
- J2 pad 17: /iCE40/S+ -> /iCE40/IO23
- J2 pad 18: /iCE40/S- -> /iCE40/IO22
- J2 pad 19: /iCE40/SCK -> /iCE40/IO25
- J2 pad 20: /iCE40/SDA -> /iCE40/IO24
- J2 pad 5: /iCE40/IO15 -> /iCE40/SDA
- J2 pad 6: /iCE40/IO16 -> /iCE40/SDA
- J2 pad 7: /iCE40/IO17 -> /iCE40/SCK
- J2 pad 8: /iCE40/IO18 -> /iCE40/SCK
- J2 pad 9: /iCE40/IO19 -> /iCE40/S+
- J7 pad 1: (no net) -> Net-(J7-Pad1)
- J7 pad 8: (no net) -> Net-(J7-Pad8)
- J8 pad 2: (no net) -> Net-(J8-Pad2)
- J8 pad 3: (no net) -> Net-(J8-Pad3)
- J8 pad 4: (no net) -> Net-(J8-Pad4)
- U1 pad 10: /iCE40/IO11 -> /iCE40/IO4
- U1 pad 11: /iCE40/IO12 -> /iCE40/IO3
- U1 pad 12: /iCE40/IO13 -> /iCE40/IO2
- U1 pad 13: /iCE40/IO15 -> /iCE40/IO1
- U1 pad 18: /iCE40/IO18 -> /iCE40/COMM3
- U1 pad 19: /iCE40/IO17 -> /iCE40/COMM2
- U1 pad 2: /iCE40/IO6 -> /iCE40/IO9
- U1 pad 20: /iCE40/IO16 -> /iCE40/COMM1
- U1 pad 21: /iCE40/IO14 -> /iCE40/COMM0
- U1 pad 23: /iCE40/IO20 -> /iCE40/RGB_R
- U1 pad 25: /iCE40/IO19 -> /iCE40/RGB_G
- U1 pad 26: /iCE40/IO22 -> /iCE40/RGB_B
- U1 pad 27: /iCE40/IO21 -> /iCE40/SDA
- U1 pad 28: /iCE40/IO23 -> /iCE40/SCK
- U1 pad 31: /iCE40/IO24 -> /iCE40/IO17
- U1 pad 32: /iCE40/IO25 -> /iCE40/IO18
- U1 pad 34: /iCE40/SCK -> /iCE40/IO19
- U1 pad 36: /iCE40/COMM0 -> /iCE40/IO20
- U1 pad 37: /iCE40/SDA -> /iCE40/IO21
- U1 pad 38: /iCE40/COMM2 -> /iCE40/IO22
- U1 pad 39: /iCE40/RGB_R -> /iCE40/IO23
- U1 pad 40: /iCE40/RGB_G -> /iCE40/IO24
- U1 pad 41: /iCE40/RGB_B -> /iCE40/IO25
- U1 pad 42: /iCE40/COMM3 -> /iCE40/IO15
- U1 pad 43: /iCE40/COMM1 -> /iCE40/IO16
- U1 pad 44: /iCE40/IO3 -> /iCE40/IO13
- U1 pad 45: /iCE40/IO5 -> /iCE40/IO14
- U1 pad 46: /iCE40/IO1 -> /iCE40/IO11
- U1 pad 47: /iCE40/IO2 -> /iCE40/IO12
- U1 pad 48: /iCE40/IO4 -> /iCE40/IO10
- U1 pad 6: /iCE40/IO9 -> /iCE40/IO6
- U1 pad 9: /iCE40/IO10 -> /iCE40/IO5
- U11 pad 24: (no net) -> Net-(U11-Pad24)
- U5 pad 13: (no net) -> Net-(U5-Pad13)
- U6 pad 15: (no net) -> Net-(U6-Pad15)
- U6 pad 16: (no net) -> Net-(U6-Pad16)
- U6 pad 17: (no net) -> Net-(U6-Pad17)
- U6 pad 18: (no net) -> Net-(U6-Pad18)
- U6 pad 19: (no net) -> Net-(U6-Pad19)
- U6 pad 20: (no net) -> Net-(U6-Pad20)
- U6 pad 21: (no net) -> Net-(U6-Pad21)
- U6 pad 22: (no net) -> Net-(U6-Pad22)
- U6 pad 23: (no net) -> Net-(U6-Pad23)
- U6 pad 24: (no net) -> Net-(U6-Pad24)
- U6 pad 25: (no net) -> Net-(U6-Pad25)
- U6 pad 7: (no net) -> Net-(U6-Pad7)

Commit message: Add files via upload
Parts:
- C1, C10, C11, C12, C13, C14, C15, C16, C17, C18, C19, C2, C20, C21, C23, C24, C25, C27, C28, C29, C3, C30, C31, C32, C33, C36, C37, C39, C4, C42, C43, C44, C47, C48, C5, C51, C52, C55, C56, C59, C60, C61, C7: footprint Capacitor_SMD:C_0603_1608Metric_Pad1.05x0.95mm_HandSolder -> Capacitor_SMD:C_0603_1608Metric
- C22, C34, C35, C40, C41, C45, C46, C49, C50, C53, C54, C57, C58: footprint Capacitor_SMD:C_0805_2012Metric_Pad1.15x1.40mm_HandSolder -> Capacitor_SMD:C_0805_2012Metric
- C38: footprint Capacitor_SMD:C_1206_3216Metric_Pad1.42x1.75mm_HandSolder -> Capacitor_SMD:C_1206_3216Metric
- C6, C8, C9: footprint Capacitor_SMD:C_0603_1608Metric_Pad1.05x0.95mm_HandSolder -> Capacitor_SMD:C_0603_1608Metric; moved to B.Cu
- D1, D10, D11, D12, D13, D2, D7, D8, D9: footprint LED_SMD:LED_0603_1608Metric_Pad1.05x0.95mm_HandSolder -> LED_SMD:LED_0603_1608Metric
- D4: footprint Diode_SMD:D_SMA_Handsoldering -> Diode_SMD:D_SMA
- J5, J6: value Conn_02x11_Odd_Even -> Conn_02x10_Odd_Even; footprint Connector_PinHeader_2.54mm:PinHeader_2x11_P2.54mm_Vertical -> Connector_PinHeader_2.54mm:PinHeader_2x10_P2.54mm_Vertical
- J7: moved to B.Cu
- L1, L2, L3, L4, L5, L6, L7, L8: footprint Inductor_SMD:L_0805_2012Metric_Pad1.15x1.40mm_HandSolder -> Inductor_SMD:L_0805_2012Metric
- R1, R100, R101, R102, R103, R104, R105, R15, R16, R2, R25, R26, R27, R3, R36, R37, R4, R5, R53, R54, R6, R88, R89, R90, R91, R92, R93, R94, R95, R96, R97, R98, R99: footprint Resistor_SMD:R_0603_1608Metric_Pad1.05x0.95mm_HandSolder -> Resistor_SMD:R_0603_1608Metric
- R46, R47, R48, R49, R50: footprint Resistor_SMD:R_0603_1608Metric_Pad1.05x0.95mm_HandSolder -> Resistor_SMD:R_0603_1608Metric; moved to F.Cu
- moved J7 106.6 mm to (54.9, 40.1), turned to 180 degrees
- moved R93 99.3 mm to (70.9, 78.0), turned to 180 degrees
- moved U10 87.0 mm to (126.7, 110.5), turned to 90 degrees
- moved R94 82.5 mm to (73.9, 78.0), turned to 180 degrees
- moved C25 61.7 mm to (128.0, 113.3)
- moved R88 51.0 mm to (122.9, 109.0), turned to 270 degrees
- moved R54 50.1 mm to (121.2, 109.0), turned to 90 degrees
- moved J5 38.5 mm to (126.8, 50.5)
- moved R2 32.6 mm to (58.4, 98.0), turned to 90 degrees
- moved D2 26.0 mm to (58.4, 94.7)
- moved J6 22.1 mm to (126.8, 79.5)
- moved R92 22.0 mm to (96.8, 68.8), turned to 270 degrees
- moved R91 19.8 mm to (98.6, 68.8), turned to 270 degrees
- moved C6 17.3 mm to (52.2, 76.5), turned to 90 degrees
- moved C8 17.2 mm to (53.8, 76.5), turned to 90 degrees
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Connections:
- J2 pad 10: /iCE40/E+ -> /iCE40/SDA
- J2 pad 12: /iCE40/S- -> /iCE40/SCK
- J2 pad 5: /iCE40/SDA -> /iCE40/S+
- J2 pad 6: /iCE40/SDA -> /iCE40/E+
- J2 pad 7: /iCE40/SCK -> /iCE40/SDA
- J2 pad 8: /iCE40/SCK -> /iCE40/S-
- J2 pad 9: /iCE40/S+ -> /iCE40/SCK
- J6 pad 1: +3V3_MCU -> /sipeedm1w/IO17
- J6 pad 10: /sipeedm1w/IO24 -> /sipeedm1w/IO26
- J6 pad 11: /sipeedm1w/IO25 -> /sipeedm1w/IO27
- J6 pad 12: /sipeedm1w/IO26 -> /sipeedm1w/IO28
- J6 pad 13: /sipeedm1w/IO27 -> /sipeedm1w/IO29
- J6 pad 14: /sipeedm1w/IO28 -> /sipeedm1w/IO30
- J6 pad 15: /sipeedm1w/IO29 -> /sipeedm1w/IO31
- J6 pad 16: /sipeedm1w/IO30 -> /sipeedm1w/IO32
- J6 pad 17: /sipeedm1w/IO31 -> /sipeedm1w/IO33
- J6 pad 18: /sipeedm1w/IO32 -> GND
- J6 pad 19: /sipeedm1w/IO33 -> +3V3_MCU
- J6 pad 2: GND -> /sipeedm1w/IO18
- J6 pad 3: +3V3_MCU -> /sipeedm1w/IO19
- J6 pad 4: GND -> /sipeedm1w/IO20
- J6 pad 5: /sipeedm1w/IO19 -> /sipeedm1w/IO21
- J6 pad 6: /sipeedm1w/IO20 -> /sipeedm1w/IO22
- J6 pad 7: /sipeedm1w/IO21 -> /sipeedm1w/IO23
- J6 pad 8: /sipeedm1w/IO22 -> /sipeedm1w/IO24
- J6 pad 9: /sipeedm1w/IO23 -> /sipeedm1w/IO25
- U1 pad 42: /iCE40/IO15 -> /iCE40/IO16
- U1 pad 43: /iCE40/IO16 -> /iCE40/IO15
- U1 pad 44: /iCE40/IO13 -> /iCE40/IO14
- U1 pad 45: /iCE40/IO14 -> /iCE40/IO13
- U1 pad 46: /iCE40/IO11 -> /iCE40/IO12
- U1 pad 47: /iCE40/IO12 -> /iCE40/IO11
- U9 pad 10: /sipeedm1w/IO29 -> /sipeedm1w/IO22
- U9 pad 11: /sipeedm1w/IO30 -> /sipeedm1w/IO21
- U9 pad 12: /sipeedm1w/IO31 -> /sipeedm1w/IO20
- U9 pad 13: /sipeedm1w/RGB_G -> /sipeedm1w/IO19
- U9 pad 14: /sipeedm1w/RGB_B -> /sipeedm1w/IO18
- U9 pad 15: /sipeedm1w/RGB_R -> /sipeedm1w/IO17
- U9 pad 16: /sipeedm1w/IO32 -> /sipeedm1w/IO16
- U9 pad 18: /sipeedm1w/IO33 -> /sipeedm1w/IO15
- U9 pad 19: /sipeedm1w/IO1 -> /sipeedm1w/IO14
- U9 pad 20: /sipeedm1w/IO2 -> /sipeedm1w/IO13
- U9 pad 21: /sipeedm1w/IO3 -> /sipeedm1w/IO12
- U9 pad 22: /sipeedm1w/IO4 -> /sipeedm1w/IO11
- U9 pad 23: /sipeedm1w/IO5 -> /sipeedm1w/IO10
- U9 pad 24: /sipeedm1w/IO6 -> /sipeedm1w/IO9
- U9 pad 25: /sipeedm1w/IO7 -> /sipeedm1w/IO8
- U9 pad 26: /sipeedm1w/SPI0_CS1 -> /sipeedm1w/IO7
- U9 pad 27: /iCE40/COMM0 -> /sipeedm1w/IO6
- U9 pad 28: /iCE40/COMM1 -> /sipeedm1w/IO5
- U9 pad 29: /iCE40/COMM2 -> /sipeedm1w/IO4
- U9 pad 30: /iCE40/COMM3 -> /sipeedm1w/IO3
- U9 pad 31: /sipeedm1w/IO8 -> /sipeedm1w/IO2
- U9 pad 32: /sipeedm1w/IO9 -> /sipeedm1w/IO1
- U9 pad 33: /sipeedm1w/IO10 -> /sipeedm1w/DVP_D2
- U9 pad 34: /sipeedm1w/IO11 -> /sipeedm1w/DVP_D1
- U9 pad 35: /sipeedm1w/IO12 -> /sipeedm1w/DVP_D3
- U9 pad 36: /sipeedm1w/IO13 -> /sipeedm1w/DVP_D0
- U9 pad 37: /sipeedm1w/IO14 -> /sipeedm1w/DVP_D4
- U9 pad 38: /sipeedm1w/IO15 -> /sipeedm1w/DVP_PCLK
- U9 pad 39: /sipeedm1w/IO16 -> /sipeedm1w/DVP_D5
- U9 pad 40: /sipeedm1w/IO17 -> /sipeedm1w/DVP_D6
- U9 pad 41: /sipeedm1w/DVP_SDA -> /sipeedm1w/DVP_XCLK
- U9 pad 42: /sipeedm1w/DVP_SCL -> /sipeedm1w/DVP_D7
- U9 pad 43: /sipeedm1w/DVP_RST -> /sipeedm1w/DVP_HSYNC
- U9 pad 44: /sipeedm1w/DVP_VSYNC -> /sipeedm1w/DVP_PWDN
- U9 pad 45: /sipeedm1w/DVP_PWDN -> /sipeedm1w/DVP_VSYNC
- U9 pad 46: /sipeedm1w/DVP_HSYNC -> /sipeedm1w/DVP_RST
- U9 pad 47: /sipeedm1w/DVP_XCLK -> /sipeedm1w/DVP_SCL
- U9 pad 48: /sipeedm1w/DVP_PCLK -> /sipeedm1w/DVP_SDA
- U9 pad 5: /sipeedm1w/IO26 -> /sipeedm1w/IO27
- U9 pad 56: /sipeedm1w/IO18 -> /sipeedm1w/RGB_R
- U9 pad 57: /sipeedm1w/IO19 -> /sipeedm1w/RGB_G
- U9 pad 58: /sipeedm1w/IO20 -> /sipeedm1w/RGB_B
- U9 pad 59: /sipeedm1w/IO21 -> /iCE40/COMM0
- U9 pad 6: /sipeedm1w/IO27 -> /sipeedm1w/IO26
- U9 pad 60: /sipeedm1w/IO22 -> /iCE40/COMM1
- U9 pad 61: /sipeedm1w/IO23 -> /iCE40/COMM2
- U9 pad 62: /sipeedm1w/IO24 -> /iCE40/COMM3
- U9 pad 63: /sipeedm1w/IO25 -> /sipeedm1w/SPI0_CS1
- U9 pad 64: /sipeedm1w/DVP_D7 -> /sipeedm1w/RX_M1
- U9 pad 65: /sipeedm1w/DVP_D6 -> /omega/RX_OM
- U9 pad 66: /sipeedm1w/DVP_D5 -> /sipeedm1w/IO28
- U9 pad 67: /sipeedm1w/DVP_D4 -> /sipeedm1w/IO29
- U9 pad 68: /sipeedm1w/DVP_D3 -> /sipeedm1w/IO30
- U9 pad 69: /sipeedm1w/DVP_D2 -> /sipeedm1w/IO31
- U9 pad 7: /sipeedm1w/RX_M1 -> /sipeedm1w/IO25
- U9 pad 70: /sipeedm1w/DVP_D1 -> /sipeedm1w/IO32
- U9 pad 71: /sipeedm1w/DVP_D0 -> /sipeedm1w/IO33
- U9 pad 8: /omega/RX_OM -> /sipeedm1w/IO24
- U9 pad 9: /sipeedm1w/IO28 -> /sipeedm1w/IO23
Routing:
- net /iCE40/CRESET_B: track 0.00 -> 118.1 mm, vias 0 -> 3
- net /iCE40/COMM0: track 0.00 -> 98.8 mm, vias 0 -> 3
- net /omega/JTAG4: track 0.00 -> 95.0 mm, vias 0 -> 2
- net /iCE40/COMM2: track 0.00 -> 93.9 mm, vias 0 -> 5
- net /iCE40/OmSPI3: track 0.00 -> 79.1 mm, vias 0 -> 2
- net /iCE40/COMM1: track 0.00 -> 75.1 mm, vias 0 -> 5
- net /sipeedm1w/SPI0_CS1: track 0.00 -> 74.5 mm, vias 0 -> 5
- net /iCE40/OmSPI2: track 0.00 -> 65.6 mm
- net /iCE40/OmSPI1: track 0.00 -> 61.0 mm, vias 0 -> 2
- net /iCE40/OmSPI0: track 0.00 -> 52.1 mm
- net /sipeedm1w/RX_M1: track 0.00 -> 48.2 mm, vias 0 -> 1
- net /sipeedm1w/IO26: track 0.00 -> 47.9 mm
- net /sipeedm1w/IO24: track 0.00 -> 46.3 mm
- net /sipeedm1w/IO32: track 0.00 -> 46.2 mm, vias 0 -> 1
- net /sipeedm1w/IO27: track 0.00 -> 45.5 mm
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Other:
- board outline added: 100 x 115 mm

Commit message: Add files via upload
Parts:
- removed C25: 0.1u, Capacitor_SMD:C_0603_1608Metric
- removed D11: BLU, LED_SMD:LED_0603_1608Metric
- removed D12, D9: GRN, LED_SMD:LED_0603_1608Metric
- removed D13: YLL, LED_SMD:LED_0603_1608Metric
- removed D7: RED, LED_SMD:LED_0603_1608Metric
- removed R100, R101, R95, R97, R99: 2k2, Resistor_SMD:R_0603_1608Metric
- removed R88: 10K, Resistor_SMD:R_0603_1608Metric
- removed U10: SMS, Connector_PinHeader_2.54mm:PinHeader_2x02_P2.54mm_Vertical
- C1, C10, C11, C12, C13, C14, C15, C16, C17, C2, C27, C28, C29, C30, C31, C32, C33, C34, C35, C36, C37, C4, C40, C41, C43, C44, C45, C46, C47, C48, C49, C50, C51, C52, C53, C54, C55, C56, C57, C58, C59, C60, C61, Q1, R15, R16, R2, R3, R5, R54, R6, R91, R92, U2, U5: moved to B.Cu
- U11: footprint Connector_FFC-FPC:Molex_502244-2430_1x24-1MP_P0.5mm_Horizontal -> Connector_FFC-FPC:Molex_502231-2400_1x24-1SH_P0.5mm_Vertical
- U14: value ZLDO1117G12TA -> XC6206P122MR; footprint Package_TO_SOT_SMD:SOT-223 -> Package_TO_SOT_SMD:SOT-23
- moved J7 56.7 mm to (102.9, 70.2)
- moved R90 38.6 mm to (51.6, 79.8)
- moved C19 38.6 mm to (44.0, 78.3)
- moved C24 38.6 mm to (58.7, 78.3)
- moved C26 38.6 mm to (51.7, 78.3)
- moved R4 38.6 mm to (44.0, 79.9)
- moved R53 38.6 mm to (58.7, 79.8), turned to 180 degrees
- moved U12 38.6 mm to (51.6, 71.9)
- moved U3 38.6 mm to (44.2, 71.8)
- moved U7 38.6 mm to (58.8, 71.7)
- moved R54 34.2 mm to (89.2, 97.0), turned to 180 degrees
- moved R93 33.6 mm to (104.1, 73.7), turned to 270 degrees
- moved D3 31.5 mm to (46.4, 87.9)
- moved R103 31.5 mm to (44.8, 81.8)
- moved R37 31.5 mm to (48.4, 81.8)
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Connections:
- J2 pad 10: /iCE40/SDA -> /iCE40/SCK
- J2 pad 12: /iCE40/SCK -> /iCE40/SDA
- J2 pad 7: /iCE40/SDA -> /iCE40/SCK
- J2 pad 9: /iCE40/SCK -> /iCE40/SDA
- U1 pad 27: /iCE40/SDA -> /iCE40/SCK
- U1 pad 28: /iCE40/SCK -> /iCE40/SDA
- U9 pad 56: /sipeedm1w/RGB_R -> /sipeedm1w/RGB_B
- U9 pad 58: /sipeedm1w/RGB_B -> /sipeedm1w/RGB_R
Routing:
- net /omega/RST: track 8.40 -> 103.4 mm, vias 0 -> 9
- net /omega/JTAG4: track 95.0 -> 36.3 mm, vias 2 -> 1
- net /iCE40/OmSPI3: track 79.1 -> 41.8 mm
- net /sipeedm1w/SPI0_CS1: track 74.5 -> 43.7 mm, vias 5 -> 1
- net /iCE40/OmSPI1: track 61.0 -> 32.7 mm, vias 2 -> 0
- net /iCE40/OmSPI0: track 52.1 -> 26.1 mm
- net /iCE40/OmSPI2: track 65.6 -> 39.7 mm, vias 0 -> 2
- net /sipeedm1w/BOOT: track 26.3 -> 5.18 mm, vias 2 -> 1
- net /iCE40/COMM0: track 98.8 -> 78.6 mm, vias 3 -> 2
- net /sipeedm1w/IO33: track 39.5 -> 57.7 mm, vias 1 -> 0
- net /sipeedm1w/IO31: track 42.8 -> 59.3 mm
- net /sipeedm1w/IO29: track 42.0 -> 58.4 mm
- net /iCE40/IO6: track 34.4 -> 18.2 mm
- net /sipeedm1w/IO30: track 45.4 -> 61.6 mm
- net GND_CASE: track 15.3 -> 0.00 mm
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Other:
- board size 100 x 115 mm -> 90 x 85 mm

Commit message: Add files via upload
Parts:
- turned C35 to 180 degrees
- turned C37 to 180 degrees
- turned C58 to 180 degrees
- turned C60 to 180 degrees
Routing:
- net +1V8_MCU: track 13.5 -> 165.5 mm, vias 2 -> 8
- net +5V: track 7.58 -> 156.7 mm, vias 1 -> 4
- net +2V8_MCU: track 1.47 -> 127.4 mm, vias 1 -> 3
- net +3V3_MCU: track 5.84 -> 131.0 mm, vias 1 -> 12
- net +1V5_MCU: track 1.78 -> 99.7 mm, vias 1 -> 5
- net +3V3_FPGA: track 20.6 -> 97.2 mm, vias 4 -> 6
- net /omega/JTAG4: track 36.3 -> 90.6 mm, vias 1 -> 5
- net +1V2_FPGA: track 9.14 -> 23.1 mm, vias 2 -> 3
- net GND_CASE: track 0.00 -> 6.22 mm
- net /sipeedm1w/IO32: track 60.8 -> 62.6 mm
- net /omega/RX_OM: track 43.0 -> 44.5 mm
- net /sipeedm1w/RX_M1: track 46.7 -> 48.2 mm
- net /omega/JTAG3: track 27.1 -> 26.6 mm
- added copper zone on B.Cu, net +1V2_FPGA
- added copper zone on B.Cu, net +1V8_MCU
- added copper zone on B.Cu, net +2V8_MCU
- added copper zone on F.Cu, net +2V8_MCU
- added copper zone on B.Cu, net +3V3_FPGA
- added copper zone on F.Cu, net +3V3_FPGA
- added copper zone on B.Cu, net +3V3_MCU
- added copper zone on B.Cu, net +5V
- added copper zone on F.Cu, net +5V
- added copper zone on F.Cu, net GND_CASE

Commit message: Add files via upload
Parts:
- moved C53 81.4 mm to (80.7, 67.9), turned to 270 degrees
- moved U17 80.8 mm to (81.5, 67.9), turned to 90 degrees
- moved C55 80.4 mm to (82.5, 67.7), turned to 270 degrees
- moved C57 79.8 mm to (84.2, 67.2), turned to 90 degrees
- moved C59 78.4 mm to (86.0, 67.4), turned to 90 degrees
- moved C47 75.2 mm to (62.0, 67.0), turned to 270 degrees
- moved C45 73.5 mm to (63.8, 67.2), turned to 270 degrees
- moved C49 71.9 mm to (65.8, 67.2), turned to 270 degrees
- moved C51 70.8 mm to (67.5, 67.0), turned to 270 degrees
- moved U15 69.0 mm to (65.6, 69.9), turned to 270 degrees
- moved D10 67.9 mm to (70.1, 67.0), turned to 90 degrees
- moved C48 66.5 mm to (73.2, 67.0), turned to 270 degrees
- moved C46 65.2 mm to (74.9, 67.2), turned to 270 degrees
- moved R98 64.4 mm to (70.1, 70.0), turned to 270 degrees
- moved C50 64.1 mm to (76.9, 67.2), turned to 270 degrees
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Routing:
- net +2V8_MCU: track 127.4 -> 3.42 mm, vias 3 -> 4
- net +1V8_MCU: track 165.5 -> 76.4 mm, vias 8 -> 10
- net +5V: track 156.7 -> 224.2 mm, vias 4 -> 16
- net +1V5_MCU: track 99.7 -> 42.6 mm
- net +3V3_MCU: track 131.0 -> 185.3 mm, vias 12 -> 20
- net +3V3_FPGA: track 97.2 -> 126.6 mm, vias 6 -> 25
- net /omega/RST: track 103.4 -> 87.7 mm, vias 9 -> 6
- net /iCE40/CRESET_B: track 114.5 -> 99.0 mm, vias 7 -> 9
- net /iCE40/OmSPI0: track 26.1 -> 38.2 mm
- net /iCE40/OmSPI2: track 39.7 -> 29.4 mm, vias 2 -> 0
- net /iCE40/OmSPI3: track 41.8 -> 32.1 mm, vias 2 -> 6
- net GND_CASE: track 6.22 -> 15.0 mm
- net GND: track 0.00 -> 8.60 mm, vias 0 -> 61
- net /iCE40/COMM2: track 81.9 -> 89.1 mm
- net Net-(J8-Pad1): track 0.00 -> 7.21 mm
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- added copper zone on B.Cu, net +1V5_MCU
- added copper zone on F.Cu, net +1V5_MCU
- added copper zone on F.Cu, net +1V8_MCU
- added copper zone on F.Cu, net +3V3_MCU
- added copper zone on B.Cu, net GND
- added copper zone on F.Cu, net GND
- added copper zone on F.Cu, net Net-(C5-Pad1)
- removed copper zone on F.Cu, net GND_CASE

Commit message: Add files via upload
Parts:
- added D7: RED, LED_SMD:LED_0603_1608Metric, F.Cu at (37.7, 139.4)
- added R95: 2k2, Resistor_SMD:R_0603_1608Metric, F.Cu at (35.4, 140.4)
- C22: moved to F.Cu
- moved R54 8.70 mm to (97.5, 106.0), turned to 270 degrees
- moved D4 4.85 mm to (108.8, 126.2)
- moved C22 2.73 mm to (107.7, 129.3)
- moved C42 2.35 mm to (37.6, 137.7)
- moved D6 1.75 mm to (59.5, 88.0)
- moved C39 1.20 mm to (37.6, 136.0)
- moved H3 1.00 mm to (119.0, 144.4)
- moved C44 0.97 mm to (42.6, 130.6)
- moved C41 0.97 mm to (42.8, 132.3)
- moved R46 0.70 mm to (65.4, 131.5)
- moved R48 0.70 mm to (65.4, 135.3)
- moved R49 0.70 mm to (65.4, 137.6)
- moved R47 0.70 mm to (65.4, 133.3)
- moved R50 0.70 mm to (65.4, 139.7)
- moved C30 0.13 mm to (82.2, 79.2)
Routing:
- net +5V: track 224.2 -> 231.9 mm, vias 16 -> 19
- net +3V3_MCU: track 185.3 -> 177.7 mm
- net Net-(C22-Pad1): track 14.6 -> 19.1 mm, vias 0 -> 1
- net /iCE40/OmSPI1: track 38.1 -> 42.6 mm
- net Net-(D5-Pad2): track 16.4 -> 12.3 mm
- net /iCE40/OmSPI2: track 29.4 -> 33.4 mm, vias 0 -> 4
- net /iCE40/CRESET_B: track 99.0 -> 102.4 mm
- net Net-(D5-Pad1): track 12.8 -> 15.8 mm
- net /sipeedm1w/BOOT: track 5.46 -> 8.21 mm
- net /iCE40/OmSPI0: track 38.2 -> 40.4 mm, vias 0 -> 2
- net +3V3_FPGA: track 126.6 -> 128.4 mm, vias 25 -> 23
- net /sipeedm1w/RGB_B: track 28.6 -> 26.8 mm, vias 0 -> 2
- net /sipeedm1w/RGB_G: track 21.5 -> 19.7 mm, vias 0 -> 2
- net +1V5_MCU: track 42.6 -> 40.8 mm, vias 5 -> 9
- net /iCE40/OmSPI3: track 32.1 -> 33.8 mm
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Other:
- board text added: "AICE"
- board text added: "JOSÉ"

Commit message: Add files via upload
Parts:
- C22: footprint Capacitor_SMD:C_0805_2012Metric -> Capacitor_THT:CP_Radial_D5.0mm_P2.00mm
