File: AICE/AICE.kicad_pcb (KiCad board)
At the start: 2 copper layers, 90 x 85 mm, 140 parts, among them J1 Conn_02x10_Odd_Even, J2 Conn_02x10_Odd_Even, J3 Conn_01x03, J4 USB_A, J5 Conn_02x10_Odd_Even, J6 Conn_02x10_Odd_Even, J7 Micro_SD_Card, J8 USB_B_Micro, Q1 S8550, U1 ICE40UP5K-SG48ITR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

Commit message: Add files via upload
Parts:
- added R7: 10K, Resistor_SMD:R_0603_1608Metric, B.Cu at (64.9, 128.6)
Routing:
- net +3V3_MCU: track 177.7 -> 174.3 mm, vias 20 -> 27
- net /iCE40/COMM1: track 76.4 -> 78.8 mm
- net /iCE40/COMM0: track 78.6 -> 80.3 mm
- net /iCE40/OmSPI2: track 33.4 -> 34.8 mm
- net /sipeedm1w/SPI0_CS1: track 48.6 -> 49.5 mm
- net +1V5_MCU: track 40.8 -> 41.5 mm
Other:
- board text added: "AICE - JG"
- board text added: "DESIGNED BY: BA"
- board text added: "MJV"
