File: AICE/_autosave-AICE.kicad_pcb (KiCad board)
At the start: 2 copper layers, 90 x 85 mm, 140 parts, among them J1 Conn_02x10_Odd_Even, J2 Conn_02x10_Odd_Even, J3 Conn_01x03, J4 USB_A, J5 Conn_02x10_Odd_Even, J6 Conn_02x10_Odd_Even, J8 USB_B_Micro, Q1 S8550, U1 ICE40UP5K-SG48ITR, U11 DVP_PORT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

Commit message: Add files via upload
Parts:
- added J7: Micro_SD_Card, Connector_Card:microSD_HC_Wuerth_693072010801, B.Cu at (102.9, 70.2)
Other:
- board size 90 x 85 mm -> 97.2 x 90.5 mm
Changed lines of the file:
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@@
   (general
     (thickness 1.6)
-    (drawings 10)
-    (tracks 2330)
+    (drawings 14)
+    (tracks 2326)
     (zones 0)
-    (modules 140)
-    (nets 170)
+    (modules 141)
+    (nets 172)
   )
   (page A4)
@@
   (net 168 "Net-(U11-Pad24)")
   (net 169 "Net-(D7-Pad1)")
+  (net 170 "Net-(J7-Pad8)")
+  (net 171 "Net-(J7-Pad1)")
   (net_class Default "This is the default net class."
     (clearance 0.2)
@@
     (add_net "Net-(J3-Pad3)")
     (add_net "Net-(J4-Pad5)")
+    (add_net "Net-(J7-Pad1)")
+    (add_net "Net-(J7-Pad8)")
     (add_net "Net-(J8-Pad1)")
     (add_net "Net-(J8-Pad2)")
@@
     )
   )
+  (module Connector_Card:microSD_HC_Wuerth_693072010801 (layer B.Cu)
+    (at 102.9 70.2 180)
+    (descr http://katalog.we-online.de/em/datasheet/693072010801.pdf)
+    (tags "Micro SD Wuerth Wurth Würth")
+    (attr smd)
+    (fp_text reference J7 (at 0 7.99) (layer B.SilkS)
+      (effects (font (size 1 1) (thickness 0.15)) (justify mirror))
+    )
+    (fp_text value Micro_SD_Card (at 0 -9.22) (layer B.Fab)
+      (effects (font (size 1 1) (thickness 0.15)) (justify mirror))
+    )
+    (fp_text user %R (at 0 -1.15) (layer B.Fab)
+      (effects (font (size 1 1) (thickness 0.15)) (justify mirror))
+    )
+    (fp_line (start -6.8 -8) (end 6.8 -8) (layer B.Fab) (width 0.1))
+    (fp_line (start -6.8 5.7) (end -6.8 -8) (layer B.Fab) (width 0.1))
+    (fp_line (start 6.8 5.7) (end -6.8 5.7) (layer B.Fab) (width 0.1))
+    (fp_line (start 6.8 -8) (end 6.8 5.7) (layer B.Fab) (width 0.1))
+    (fp_line (start 5 6.61) (end 5.5 6.71) (layer B.SilkS) (width 0.12))
+    (fp_line (start 3.7 6.31) (end 5 6.61) (layer B.SilkS) (width 0.12))
+    (fp_line (start 2.2 6.11) (end 3.7 6.31) (layer B.SilkS) (width 0.12))
+    (fp_line (start 0.9 6.01) (end 2.2 6.11) (layer B.SilkS) (width 0.12))
+    (fp_line (start -0.9 6.01) (end 0.9 6.01) (layer B.SilkS) (width 0.12))
+    (fp_line (start -2.2 6.11) (end -0.9 6.01) (layer B.SilkS) (width 0.12))
+    (fp_line (start -3 6.21) (end -2.2 6.11) (layer B.SilkS) (width 0.12))
+    (fp_line (start -4.7 6.51) (end -3 6.21) (layer B.SilkS) (width 0.12))
+    (fp_line (start -5.5 6.71) (end -4.7 6.51) (layer B.SilkS) (width 0.12))
+    (fp_line (start -5 7.31) (end 5 7.31) (layer B.SilkS) (width 0.12))
+    (fp_line (start -5.5 5.81) (end -5.5 6.81) (layer B.SilkS) (width 0.12))
+    (fp_line (start 5.5 5.81) (end 5.5 6.81) (layer B.SilkS) (width 0.12))
+    (fp_line (start -6.91 5.81) (end 6.91 5.81) (layer B.SilkS) (width 0.12))
+    (fp_line (start 6.91 -8.11) (end -6.91 -8.11) (layer B.SilkS) (width 0.12))
+    (fp_line (start 6.91 -5.41) (end 6.91 -8.11) (layer B.SilkS) (width 0.12))
+    (fp_line (start 6.91 5.81) (end 6.91 5.41) (layer B.SilkS) (width 0.12))
+    (fp_line (start 6.91 2.89) (end 6.91 -2.89) (layer B.SilkS) (width 0.12))
+    (fp_line (start -6.91 -5.41) (end -6.91 -8.11) (layer B.SilkS) (width 0.12))
+    (fp_line (start -6.91 2.89) (end -6.91 -2.89) (layer B.SilkS) (width 0.12))
+    (fp_line (start -6.91 5.81) (end -6.91 5.41) (layer B.SilkS) (width 0.12))
+    (fp_line (start 8.08 6.2) (end 8.08 -8.5) (layer B.CrtYd) (width 0.05))
+    (fp_line (start 8.08 6.2) (end -8.08 6.2) (layer B.CrtYd) (width 0.05))
+    (fp_line (start 8.08 -8.5) (end -8.08 -8.5) (layer B.CrtYd) (width 0.05))
+    (fp_line (start -8.08 6.2) (end -8.08 -8.5) (layer B.CrtYd) (width 0.05))
+    (fp_arc (start 5 6.81) (end 5 7.31) (angle -90) (layer B.SilkS) (width 0.12))
+    (fp_arc (start -5 6.81) (end -5.5 6.81) (angle -90) (layer B.SilkS) (width 0.12))
+    (pad 9 smd rect (at 6.875 4.15 180) (size 1.45 2) (layers B.Cu B.Paste B.Mask)
+      (net 2 GND))
+    (pad 9 smd rect (at -6.875 4.15 180) (size 1.45 2) (layers B.Cu B.Paste B.Mask)
+      (net 2 GND))
+    (pad 9 smd rect (at -6.875 -4.15 180) (size 1.45 2) (layers B.Cu B.Paste B.Mask)
+      (net 2 GND))
+    (pad 9 smd rect (at 6.875 -4.15 180) (size 1.45 2) (layers B.Cu B.Paste B.Mask)
+      (net 2 GND))
+    (pad 8 smd rect (at 4.5 1.55 180) (size 0.8 1.5) (layers B.Cu B.Paste B.Mask)
+      (net 170 "Net-(J7-Pad8)"))
+    (pad 7 smd rect (at 3.4 1.55 180) (size 0.8 1.5) (layers B.Cu B.Paste B.Mask)
+      (net 114 /iCE40/COMM0))
+    (pad 6 smd rect (at 2.3 1.55 180) (size 0.8 1.5) (layers B.Cu B.Paste B.Mask)
+      (net 2 GND))
+    (pad 5 smd rect (at 1.2 1.55 180) (size 0.8 1.5) (layers B.Cu B.Paste B.Mask)
+      (net 117 /iCE40/COMM1))
+    (pad 4 smd rect (at 0.1 1.55 180) (size 0.8 1.5) (layers B.Cu B.Paste B.Mask)
+      (net 10 +3V3_MCU))
+    (pad 3 smd rect (at -1 1.55 180) (size 0.8 1.5) (layers B.Cu B.Paste B.Mask)
+      (net 115 /iCE40/COMM2))
+    (pad 2 smd rect (at -2.1 1.55 180) (size 0.8 1.5) (layers B.Cu B.Paste B.Mask)
+      (net 99 /sipeedm1w/SPI0_CS1))
+    (pad 1 smd rect (at -3.2 1.55 180) (size 0.8 1.5) (layers B.Cu B.Paste B.Mask)
+      (net 171 "Net-(J7-Pad1)"))
+    (model ${KISYS3DMOD}/Connector_Card.3dshapes/microSD_HC_Wuerth_693072010801.wrl
+      (at (xyz 0 0 0))
+      (scale (xyz 1 1 1))
+      (rotate (xyz 0 0 0))
+    )
+  )
+  (gr_line (start 126.8 60.7) (end 126.95 151.25) (layer Edge.Cuts) (width 0.1))
+  (gr_line (start 29.8 60.7) (end 126.8 60.7) (layer Edge.Cuts) (width 0.1))
+  (gr_line (start 29.85 151.25) (end 29.8 60.7) (layer Edge.Cuts) (width 0.1))
+  (gr_line (start 126.95 151.25) (end 29.85 151.25) (layer Edge.Cuts) (width 0.1))
   (gr_text MJV (at 102.3 107.65) (layer F.SilkS)
     (effects (font (size 1 1) (thickness 0.25)))
@@
   (segment (start 94.6 77.65) (end 95.599994 77.65) (width 0.6) (layer F.Cu) (net 10))
   (segment (start 96.5 77.65) (end 95.599994 77.65) (width 0.6) (layer F.Cu) (net 10))
-  (segment (start 88.1 81.9) (end 88.1 81.9) (width 0.6) (layer B.Cu) (net 10))
   (segment (start 88.7 81.3) (end 89.3 80.7) (width 0.6) (layer B.Cu) (net 10))
   (segment (start 89.3 80.7) (end 88.7 81.3) (width 0.6) (layer F.Cu) (net 10))
-  (segment (start 88.1 81.9) (end 88.1 81.9) (width 0.6) (layer F.Cu) (net 10))
   (via (at 88.7 81.3) (size 0.8) (drill 0.4) (layers F.Cu B.Cu) (net 10))
   (segment (start 88.7 81.3) (end 88.12501 81.87499) (width 0.6) (layer B.Cu) (net 10))
@@
   (segment (start 81.3 82) (end 79.95 82) (width 0.6) (layer B.Cu) (net 10))
   (via (at 81.3 82) (size 0.8) (drill 0.4) (layers F.Cu B.Cu) (net 10))
-  (segment (start 79.95 82) (end 79.95 82) (width 0.6) (layer B.Cu) (net 10))
   (segment (start 79.684315 82) (end 80.15 82) (width 0.6) (layer F.Cu) (net 10))
   (segment (start 79.670713 82.013602) (end 79.684315 82) (width 0.6) (layer F.Cu) (net 10))
@@
   (segment (start 85.65 81.9) (end 85.55 82) (width 0.6) (layer F.Cu) (net 10))
   (segment (start 85.55 82) (end 84.6 82) (width 0.6) (layer F.Cu) (net 10))
-  (segment (start 84.6 82) (end 84.6 82) (width 0.6) (layer F.Cu) (net 10))
   (via (at 84.6 82) (size 0.8) (drill 0.4) (layers F.Cu B.Cu) (net 10))
   (segment (start 84.6 82) (end 81.3 82) (width 0.6) (layer B.Cu) (net 10))
@@
   (segment (start 79.652094 81.113601) (end 79.086409 81.113601) (width 0.6) (layer B.Cu) (net 16))
   (segment (start 85.68944 80.44506) (end 85.034501 81.099999) (width 0.6) (layer B.Cu) (net 16))
-  (segment (start 85.68944 80.00756) (end 85.68944 80.44506) (width 0.6) (layer B.Cu) (net 16))
+  (segment (start 85.68944 80.00756) (end 85.68944 80.44506) (width 0.6) (layer B.Cu) (net 16) (status 10))
   (segment (start 63.28482 66.75612) (end 63.28482 66.50612) (width 1) (layer F.Cu) (net 17) (status 30))
   (segment (start 42.077878 64.75612) (end 40.366001 66.467997) (width 1) (layer F.Cu) (net 17))
@@
   (segment (start 45.396 104.638) (end 45.396 105.765589) (width 0.25) (layer B.Cu) (net 113) (status 10))
   (via (at 92.3925 79.88046) (size 0.8) (drill 0.4) (layers F.Cu B.Cu) (net 114))
-  (segment (start 99.51 69.65) (end 99.51 68.65) (width 0.25) (layer B.Cu) (net 114) (status 20))
+  (segment (start 99.51 69.65) (end 99.51 68.65) (width 0.25) (layer B.Cu) (net 114))
   (segment (start 103.47198 72.65152) (end 100.15152 72.65152) (width 0.25) (layer F.Cu) (net 114) (status 10))
   (segment (start 99.5 72) (end 99.51 69.65) (width 0.25) (layer B.Cu) (net 114))
@@
   (segment (start 85.15 84.2) (end 87.025887 84.2) (width 0.25) (layer F.Cu) (net 114))
   (via (at 95.07474 80.89646) (size 0.8) (drill 0.4) (layers F.Cu B.Cu) (net 115))
-  (segment (start 103.91 69.65) (end 103.91 68.65) (width 0.25) (layer B.Cu) (net 115) (status 20))
+  (segment (start 103.91 69.65) (end 103.91 68.65) (width 0.25) (layer B.Cu) (net 115))
   (via (at 105.3 70.7) (size 0.8) (drill 0.4) (layers F.Cu B.Cu) (net 115))
   (segment (start 104.25 69.65) (end 103.91 69.65) (width 0.25) (layer B.Cu) (net 115))
@@
   (segment (start 61.45 128.6) (end 60.95 128.1) (width 0.25) (layer F.Cu) (net 151))
   (segment (start 62.7 128.6) (end 61.45 128.6) (width 0.25) (layer F.Cu) (net 151))
-  (segment (start 62.7 128.6) (end 64.1125 128.6) (width 0.25) (layer B.Cu) (net 151))
+  (segment (start 62.7 128.6) (end 64.1125 128.6) (width 0.25) (layer B.Cu) (net 151) (status 20))
   (segment (start 35.5625 139.45) (end 35.35 139.6625) (width 0.25) (layer F.Cu) (net 169) (status 30))
   (segment (start 36.875 139.45) (end 35.5625 139.45) (width 0.25) (layer F.Cu) (net 169) (status 30))
